File: rfm12_rfm01_breakout/rfm12_rfm01_breakout.sch (KiCad schematic (older format))
At the start: 13 parts, among them J1 ANT, J2 CONN_01X07, U1 RFM12B

Commit message: Forgot to commit some changes
Parts:
- gave numbers to parts that had none: 1
Changed lines of the file:
@@
 $EndComp
 $Comp
-L GND #PWR01
+L GND #PWR2
 U 1 1 59A2C161
 P 5450 3150
-F 0 "#PWR01" H 5450 2900 50  0001 C CNN
+F 0 "#PWR2" H 5450 2900 50  0001 C CNN
 F 1 "GND" V 5450 2950 50  0000 C CNN
 F 2 "" H 5450 3150 50  0001 C CNN
@@
 $EndComp
 $Comp
-L +3.3V #PWR02
+L +3.3V #PWR3
 U 1 1 59A2C191
 P 5450 3250
-F 0 "#PWR02" H 5450 3100 50  0001 C CNN
+F 0 "#PWR3" H 5450 3100 50  0001 C CNN
 F 1 "+3.3V" V 5450 3450 50  0000 C CNN
 F 2 "" H 5450 3250 50  0001 C CNN
@@
 Connection ~ 5600 3850
 $Comp
-L GND #PWR03
+L GND #PWR4
 U 1 1 59A2C410
 P 5600 4100
-F 0 "#PWR03" H 5600 3850 50  0001 C CNN
+F 0 "#PWR4" H 5600 3850 50  0001 C CNN
 F 1 "GND" H 5600 3950 50  0000 C CNN
 F 2 "" H 5600 4100 50  0001 C CNN
@@
 $EndComp
 $Comp
-L GND #PWR04
+L GND #PWR7
 U 1 1 59A2C434
 P 6000 4100
-F 0 "#PWR04" H 6000 3850 50  0001 C CNN
+F 0 "#PWR7" H 6000 3850 50  0001 C CNN
 F 1 "GND" H 6000 3950 50  0000 C CNN
 F 2 "" H 6000 4100 50  0001 C CNN
@@
 MISO
 $Comp
-L GND #PWR05
+L GND #PWR1
 U 1 1 59A2C654
 P 3750 3350
-F 0 "#PWR05" H 3750 3100 50  0001 C CNN
+F 0 "#PWR1" H 3750 3100 50  0001 C CNN
 F 1 "GND" V 3750 3150 50  0000 C CNN
 F 2 "" H 3750 3350 50  0001 C CNN
@@
 $EndComp
 $Comp
-L GND #PWR06
+L GND #PWR6
 U 1 1 59A2CB99
 P 5900 3100
-F 0 "#PWR06" H 5900 2850 50  0001 C CNN
+F 0 "#PWR6" H 5900 2850 50  0001 C CNN
 F 1 "GND" H 5900 2950 50  0000 C CNN
 F 2 "" H 5900 3100 50  0001 C CNN
@@
 $EndComp
 $Comp
-L +3.3V #PWR07
+L +3.3V #PWR5
 U 1 1 59A2CBC5
 P 5900 2900
-F 0 "#PWR07" H 5900 2750 50  0001 C CNN
+F 0 "#PWR5" H 5900 2750 50  0001 C CNN
 F 1 "+3.3V" H 5900 3040 50  0000 C CNN
 F 2 "" H 5900 2900 50  0001 C CNN
@@
 $EndComp
 $Comp
-L +3.3V #PWR08
+L +3.3V #PWR9
 U 1 1 59A2D105
 P 6750 3250
-F 0 "#PWR08" H 6750 3100 50  0001 C CNN
+F 0 "#PWR9" H 6750 3100 50  0001 C CNN
 F 1 "+3.3V" V 6750 3450 50  0000 C CNN
 F 2 "" H 6750 3250 50  0001 C CNN
@@
 $EndComp
 $Comp
-L GND #PWR09
+L GND #PWR8
 U 1 1 59A2D134
 P 6750 3150
-F 0 "#PWR09" H 6750 2900 50  0001 C CNN
+F 0 "#PWR8" H 6750 2900 50  0001 C CNN
 F 1 "GND" V 6750 2950 50  0000 C CNN
 F 2 "" H 6750 3150 50  0001 C CNN
@@
 $EndComp
 $Comp
-L CONN_01X01 J?
+L CONN_01X01 J3
 U 1 1 59A2D446
 P 6700 3650
-F 0 "J?" H 6700 3750 50  0000 C CNN
+F 0 "J3" H 6700 3750 50  0000 C CNN
 F 1 "INT" V 6800 3650 50  0000 C CNN
 F 2 "Pin_Headers:Pin_Header_Straight_1x01_Pitch2.54mm" H 6700 3650 50  0001 C CNN
