File: atmega_isp_programming/atmega_isp_programming.kicad_pcb (KiCad board)
At the start: 2 copper layers, 19.2 x 15.3 mm, 3 parts, among them P1 CONN_02X03, P2 CONN_01X06

Commit message: Updated footprint for SPI connector
Parts:
- moved C1 12.1 mm to (143.6, 108.1), turned to 180 degrees
- moved P1 1.50 mm to (152.2, 103.3)
Connections:
- P2 pad 1: +3V3 -> MOSI
- P2 pad 2: GND -> MISO
- P2 pad 3: MOSI -> CLK
- P2 pad 4: MISO -> CS
- P2 pad 5: CLK -> +3V3
- P2 pad 6: CS -> GND
Routing:
- net GND: track 0.00 -> 10.8 mm, vias 0 -> 3
- net MOSI: track 5.32 -> 11.1 mm
- net CLK: track 11.0 -> 8.02 mm
- net MISO: track 10.1 -> 8.03 mm
- net CS: track 9.75 -> 8.59 mm
Changed lines of the file:
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@@
-(kicad_pcb (version 4) (host pcbnew 4.0.4-stable)
+(kicad_pcb (version 4) (host pcbnew 4.0.6)
   (general
     (links 8)
-    (no_connects 6)
-    (area 138.99 99.436666 160.075001 118.200001)
+    (no_connects 8)
+    (area 140.674999 101.424999 160.075001 116.875001)
     (thickness 1.6)
     (drawings 10)
-    (tracks 26)
+    (tracks 29)
     (zones 0)
     (modules 3)
@@
   )
   (module Capacitors_SMD:C_0805_HandSoldering (layer F.Cu)
-    (at 155.65 108.2)
+    (at 143.55 108.1 180)
     (descr "Capacitor SMD 0805, hand soldering")
     (tags "capacitor 0805")
     (attr smd)
-    (fp_text reference C1 (at 0 -1.75) (layer F.SilkS) hide
-      (effects (font (size 1 1) (thickness 0.15)))
-    )
-    (fp_text value C_Small (at 0 1.75) (layer F.Fab) hide
-      (effects (font (size 1 1) (thickness 0.15)))
-    )
-    (fp_text user %R (at 0 -1.75) (layer F.Fab) hide
+    (fp_text reference C1 (at 0 -1.75 180) (layer F.SilkS) hide
+      (effects (font (size 1 1) (thickness 0.15)))
+    )
+    (fp_text value C_Small (at 0 1.75 180) (layer F.Fab) hide
+      (effects (font (size 1 1) (thickness 0.15)))
+    )
+    (fp_text user %R (at 0 -1.75 180) (layer F.Fab) hide
       (effects (font (size 1 1) (thickness 0.15)))
     )
@@
     (fp_line (start 2.25 0.87) (end 2.25 -0.88) (layer F.CrtYd) (width 0.05))
     (fp_line (start 2.25 0.87) (end -2.25 0.87) (layer F.CrtYd) (width 0.05))
-    (pad 1 smd rect (at -1.25 0) (size 1.5 1.25) (layers F.Cu F.Paste F.Mask)
+    (pad 1 smd rect (at -1.25 0 180) (size 1.5 1.25) (layers F.Cu F.Paste F.Mask)
       (net 1 +3V3))
-    (pad 2 smd rect (at 1.25 0) (size 1.5 1.25) (layers F.Cu F.Paste F.Mask)
+    (pad 2 smd rect (at 1.25 0 180) (size 1.5 1.25) (layers F.Cu F.Paste F.Mask)
       (net 2 GND))
     (model Capacitors_SMD.3dshapes/C_0805.wrl
@@
     )
     (pad 1 thru_hole rect (at 0 0 270) (size 1.7 1.7) (drill 1) (layers *.Cu *.Mask)
+      (net 6 MOSI))
+    (pad 2 thru_hole oval (at 0 2.54 270) (size 1.7 1.7) (drill 1) (layers *.Cu *.Mask)
+      (net 4 MISO))
+    (pad 3 thru_hole oval (at 0 5.08 270) (size 1.7 1.7) (drill 1) (layers *.Cu *.Mask)
+      (net 5 CLK))
+    (pad 4 thru_hole oval (at 0 7.62 270) (size 1.7 1.7) (drill 1) (layers *.Cu *.Mask)
+      (net 3 CS))
+    (pad 5 thru_hole oval (at 0 10.16 270) (size 1.7 1.7) (drill 1) (layers *.Cu *.Mask)
       (net 1 +3V3))
-    (pad 2 thru_hole oval (at 0 2.54 270) (size 1.7 1.7) (drill 1) (layers *.Cu *.Mask)
+    (pad 6 thru_hole oval (at 0 12.7 270) (size 1.7 1.7) (drill 1) (layers *.Cu *.Mask)
       (net 2 GND))
-    (pad 3 thru_hole oval (at 0 5.08 270) (size 1.7 1.7) (drill 1) (layers *.Cu *.Mask)
-      (net 6 MOSI))
-    (pad 4 thru_hole oval (at 0 7.62 270) (size 1.7 1.7) (drill 1) (layers *.Cu *.Mask)
-      (net 4 MISO))
-    (pad 5 thru_hole oval (at 0 10.16 270) (size 1.7 1.7) (drill 1) (layers *.Cu *.Mask)
-      (net 5 CLK))
-    (pad 6 thru_hole oval (at 0 12.7 270) (size 1.7 1.7) (drill 1) (layers *.Cu *.Mask)
-      (net 3 CS))
     (model ${KISYS3DMOD}/Pin_Headers.3dshapes/Pin_Header_Straight_1x06_Pitch2.54mm.wrl
       (at (xyz 0 -0.25 0))
@@
   )
   (module Pin_Headers:Pin_Header_Straight_2x03_Pitch2.54mm (layer F.Cu)
-    (at 150.74 103.2 270)
+    (at 152.24 103.3 270)
     (descr "Through hole straight pin header, 2x03, 2.54mm pitch, double rows")
     (tags "Through hole pin header THT 2x03 2.54mm double row")
@@
   (gr_line (start 140.75 101.5) (end 156.75 101.5) (layer Edge.Cuts) (width 0.15))
   (gr_line (start 140.75 111.75) (end 140.75 101.5) (layer Edge.Cuts) (width 0.15))
-  (segment (start 151 106) (end 150.74 105.74) (width 0.4) (layer F.Cu) (net 1))
-  (segment (start 152.25 107.8) (end 153.695 107.8) (width 0.4) (layer F.Cu) (net 1))
-  (segment (start 152.25 107.8) (end 152.05 107.8) (width 0.4) (layer F.Cu) (net 1))
-  (segment (start 150.74 105.74) (end 150.74 106.942081) (width 0.4) (layer F.Cu) (net 1))
-  (segment (start 150.74 106.942081) (end 151.597919 107.8) (width 0.4) (layer F.Cu) (net 1))
-  (segment (start 151.597919 107.8) (end 153.695 107.8) (width 0.4) (layer F.Cu) (net 1))
-  (segment (start 153.695 107.8) (end 154.995 109.1) (width 0.4) (layer F.Cu) (net 1))
-  (segment (start 154.995 109.1) (end 154.995 110.35) (width 0.4) (layer F.Cu) (net 1))
-  (segment (start 150.74 105.74) (end 150.74 106.51) (width 0.4) (layer F.Cu) (net 1))
-  (segment (start 154.95 110.305) (end 154.995 110.35) (width 0.4) (layer F.Cu) (net 1))
-  (segment (start 143.6 103.2) (end 142.295 104.505) (width 0.25) (layer F.Cu) (net 3))
-  (segment (start 142.295 104.505) (end 142.295 110.35) (width 0.25) (layer F.Cu) (net 3))
-  (segment (start 145.66 103.2) (end 143.6 103.2) (width 0.25) (layer F.Cu) (net 3))
-  (segment (start 150.74 103.2) (end 149.5 104.44) (width 0.25) (layer B.Cu) (net 4))
-  (segment (start 149.5 104.44) (end 147.36 104.44) (width 0.25) (layer B.Cu) (net 4))
-  (segment (start 147.36 104.44) (end 146.95 104.85) (width 0.25) (layer B.Cu) (net 4))
-  (segment (start 146.95 104.85) (end 146.95 109.925) (width 0.25) (layer B.Cu) (net 4))
-  (segment (start 146.95 109.925) (end 147.375 110.35) (width 0.25) (layer B.Cu) (net 4))
-  (segment (start 144.835 110.35) (end 144.835 109.147919) (width 0.25) (layer F.Cu) (net 5))
-  (segment (start 144.835 109.147919) (end 143.6 107.912919) (width 0.25) (layer F.Cu) (net 5))
-  (segment (start 143.6 107.912919) (end 143.6 105.3) (width 0.25) (layer F.Cu) (net 5))
-  (segment (start 143.6 105.3) (end 144.45 104.45) (width 0.25) (layer F.Cu) (net 5))
-  (segment (start 144.45 104.45) (end 146.95 104.45) (width 0.25) (layer F.Cu) (net 5))
-  (segment (start 146.95 104.45) (end 148.2 103.2) (width 0.25) (layer F.Cu) (net 5))
-  (segment (start 148.2 105.74) (end 148.2 108.635) (width 0.25) (layer B.Cu) (net 6))
-  (segment (start 148.2 108.635) (end 149.915 110.35) (width 0.25) (layer B.Cu) (net 6))
+  (segment (start 144.8 108.1) (end 149.98 108.1) (width 0.4) (layer F.Cu) (net 1))
+  (segment (start 149.98 108.1) (end 152.24 105.84) (width 0.4) (layer F.Cu) (net 1))
+  (segment (start 144.835 110.35) (end 144.835 108.135) (width 0.4) (layer F.Cu) (net 1))
+  (segment (start 144.835 108.135) (end 144.8 108.1) (width 0.4) (layer F.Cu) (net 1))
+  (segment (start 149.75 108.8) (end 152.4 108.8) (width 0.25) (layer F.Cu) (net 2))
+  (segment (start 152.4 108.8) (end 152.425 108.775) (width 0.25) (layer F.Cu) (net 2))
+  (via (at 152.425 108.775) (size 0.6) (drill 0.4) (layers F.Cu B.Cu) (net 2))
+  (segment (start 146.4 108.825) (end 149.725 108.825) (width 0.25) (layer F.Cu) (net 2))
+  (segment (start 149.725 108.825) (end 149.75 108.8) (width 0.25) (layer F.Cu) (net 2))
+  (via (at 149.75 108.8) (size 0.6) (drill 0.4) (layers F.Cu B.Cu) (net 2))
+  (segment (start 142.295 110.35) (end 143.82 108.825) (width 0.25) (layer B.Cu) (net 2))
+  (segment (start 143.82 108.825) (end 146.4 108.825) (width 0.25) (layer B.Cu) (net 2))
+  (via (at 146.4 108.825) (size 0.6) (drill 0.4) (layers F.Cu B.Cu) (net 2))
+  (segment (start 148.4 109.325) (end 148.4 104.54) (width 0.25) (layer B.Cu) (net 3))
+  (segment (start 148.4 104.54) (end 147.16 103.3) (width 0.25) (layer B.Cu) (net 3))
+  (segment (start 147.375 110.35) (end 148.4 109.325) (width 0.25) (layer B.Cu) (net 3))
+  (segment (start 146.95 109.925) (end 147.375 110.35) (width 0.25) (layer B.Cu) (net 3))
+  (segment (start 152.455 110.35) (end 153.525 109.28) (width 0.25) (layer B.Cu) (net 4))
+  (segment (start 153.525 109.28) (end 153.525 104.6) (width 0.25) (layer B.Cu) (net 4))
+  (segment (start 153.525 104.6) (end 152.24 103.315) (width 0.25) (layer B.Cu) (net 4))
+  (segment (start 152.24 103.315) (end 152.24 103.3) (width 0.25) (layer B.Cu) (net 4))
+  (segment (start 150.975 109.29) (end 150.975 104.575) (width 0.25) (layer B.Cu) (net 5))
+  (segment (start 150.975 104.575) (end 149.7 103.3) (width 0.25) (layer B.Cu) (net 5))
+  (segment (start 149.915 110.35) (end 150.975 109.29) (width 0.25) (layer B.Cu) (net 5))
+  (segment (start 154 104.575) (end 154.995 105.57) (width 0.25) (layer F.Cu) (net 6))
+  (segment (start 154.995 105.57) (end 154.995 110.35) (width 0.25) (layer F.Cu) (net 6))
+  (segment (start 150.965 104.575) (end 154 104.575) (width 0.25) (layer F.Cu) (net 6))
+  (segment (start 149.7 105.84) (end 150.965 104.575) (width 0.25) (layer F.Cu) (net 6))
+  (segment (start 154.95 110.305) (end 154.995 110.35) (width 0.4) (layer F.Cu) (net 6))
   (zone (net 2) (net_name GND) (layer F.Cu) (hatch edge 0.508)
     (connect_pads (clearance 0.3))
