File: atmega_isp_programming/atmega_isp_programming.sch (KiCad schematic (older format))
At the start: 3 parts, among them P1 CONN_02X03, P2 CONN_01X06

Commit message: Updated footprint for SPI connector
Connections:
- net +3V3: now also P2.5 (P5); no longer P2.1 (P1)
- net CLK: now also P2.3 (P3); no longer P2.5 (P5)
- net CS: now also P2.4 (P4); no longer P2.6 (P6)
- net GND: now also P2.6 (P6); no longer P2.2 (P2)
- net MISO: now also P2.2 (P2); no longer P2.4 (P4)
- net MOSI: now also P2.1 (P1); no longer P2.3 (P3)
Changed lines of the file:
@@
 L +3.3V #PWR01
 U 1 1 590E98A4
-P 5850 2950
-F 0 "#PWR01" H 5850 2800 50  0001 C CNN
-F 1 "+3.3V" V 5850 3200 50  0000 C CNN
-F 2 "" H 5850 2950 50  0000 C CNN
-F 3 "" H 5850 2950 50  0000 C CNN
-	1    5850 2950
+P 5850 3350
+F 0 "#PWR01" H 5850 3200 50  0001 C CNN
+F 1 "+3.3V" V 5850 3600 50  0000 C CNN
+F 2 "" H 5850 3350 50  0000 C CNN
+F 3 "" H 5850 3350 50  0000 C CNN
+	1    5850 3350
 	0    -1   -1   0
 $EndComp
@@
 L GND #PWR02
 U 1 1 590E98E4
-P 5850 3050
-F 0 "#PWR02" H 5850 2800 50  0001 C CNN
-F 1 "GND" V 5850 2850 50  0000 C CNN
-F 2 "" H 5850 3050 50  0000 C CNN
-F 3 "" H 5850 3050 50  0000 C CNN
-	1    5850 3050
+P 5850 3450
+F 0 "#PWR02" H 5850 3200 50  0001 C CNN
+F 1 "GND" V 5850 3250 50  0000 C CNN
+F 2 "" H 5850 3450 50  0000 C CNN
+F 3 "" H 5850 3450 50  0000 C CNN
+	1    5850 3450
 	0    1    1    0
 $EndComp
+Text GLabel 5850 2950 0    60   Input ~ 0
+MOSI
+Text GLabel 5850 3050 0    60   Input ~ 0
+MISO
 Text GLabel 5850 3150 0    60   Input ~ 0
-MOSI
+CLK
 Text GLabel 5850 3250 0    60   Input ~ 0
-MISO
-Text GLabel 5850 3350 0    60   Input ~ 0
-CLK
-Text GLabel 5850 3450 0    60   Input ~ 0
 CS
 $Comp
