File: tp4056_usb_board/tp4056_breakout.sch (KiCad schematic (older format))
At the start: 22 parts, among them J1 USB_OTG, J2 TP4056, J3 DW01, J4 8205A, J5 TEST_2P, U1 TP4056_BREAKOUT, U2 CP2102N-20P

Commit message: Changed layout/UART header for the new back board
Connections:
- net RST: now also RN1.1 (R1.1); no longer RN1.4 (R4.1)
- net RX_LED: now also RN1.4 (R4.1); no longer RN1.2 (R2.1)
- net TX_LED: now also RN1.3 (R3.1); no longer RN1.1 (R1.1)
- net VDD: now also RN1.8 (R1.2); no longer RN1.5 (R4.2)
- net at RN1.6 (R3.2): now also D4.1 (K)
- net at D3.1 (K): now also RN1.5 (R4.2); no longer RN1.7 (R2.2)
Other:
- moved on the sheet: D3, D4
Changed lines of the file:
@@
 $EndComp
 $Comp
-L VSS #PWR19
+L VSS #PWR01
 U 1 1 595C1537
 P 5750 2400
-F 0 "#PWR19" H 5750 2250 50  0001 C CNN
+F 0 "#PWR01" H 5750 2250 50  0001 C CNN
 F 1 "VSS" V 5750 2600 50  0000 C CNN
 F 2 "" H 5750 2400 50  0001 C CNN
@@
 NoConn ~ 3850 1650
 $Comp
-L GND #PWR3
+L GND #PWR02
 U 1 1 595C168E
 P 3450 1850
-F 0 "#PWR3" H 3450 1600 50  0001 C CNN
+F 0 "#PWR02" H 3450 1600 50  0001 C CNN
 F 1 "GND" H 3400 1700 50  0000 C CNN
 F 2 "" H 3450 1850 50  0001 C CNN
@@
 $EndComp
 $Comp
-L GND #PWR4
+L GND #PWR03
 U 1 1 595C16C7
 P 3550 1850
-F 0 "#PWR4" H 3550 1600 50  0001 C CNN
+F 0 "#PWR03" H 3550 1600 50  0001 C CNN
 F 1 "GND" H 3600 1700 50  0000 C CNN
 F 2 "" H 3550 1850 50  0001 C CNN
@@
 $EndComp
 $Comp
-L GND #PWR18
+L GND #PWR04
 U 1 1 595C1A34
 P 5500 3300
-F 0 "#PWR18" H 5500 3050 50  0001 C CNN
+F 0 "#PWR04" H 5500 3050 50  0001 C CNN
 F 1 "GND" H 5500 3150 50  0000 C CNN
 F 2 "" H 5500 3300 50  0001 C CNN
@@
 $EndComp
 $Comp
-L GND #PWR12
+L GND #PWR05
 U 1 1 595C1C7D
 P 4900 3700
-F 0 "#PWR12" H 4900 3450 50  0001 C CNN
+F 0 "#PWR05" H 4900 3450 50  0001 C CNN
 F 1 "GND" V 4850 3500 50  0000 C CNN
 F 2 "" H 4900 3700 50  0001 C CNN
@@
 $EndComp
 $Comp
-L +5V #PWR5
+L +5V #PWR06
 U 1 1 595C216B
 P 3900 1150
-F 0 "#PWR5" H 3900 1000 50  0001 C CNN
+F 0 "#PWR06" H 3900 1000 50  0001 C CNN
 F 1 "+5V" H 3900 1290 50  0000 C CNN
 F 2 "" H 3900 1150 50  0001 C CNN
@@
 $EndComp
 $Comp
-L +5V #PWR21
+L +5V #PWR07
 U 1 1 595C21FD
 P 6000 3800
-F 0 "#PWR21" H 6000 3650 50  0001 C CNN
+F 0 "#PWR07" H 6000 3650 50  0001 C CNN
 F 1 "+5V" H 6000 3940 50  0000 C CNN
 F 2 "" H 6000 3800 50  0001 C CNN
@@
 $EndComp
 $Comp
-L +5V #PWR16
+L +5V #PWR08
 U 1 1 595C2374
 P 5400 3700
-F 0 "#PWR16" H 5400 3550 50  0001 C CNN
+F 0 "#PWR08" H 5400 3550 50  0001 C CNN
 F 1 "+5V" V 5400 3900 50  0000 C CNN
 F 2 "" H 5400 3700 50  0001 C CNN
@@
 $EndComp
 $Comp
-L +5V #PWR11
+L +5V #PWR09
 U 1 1 595C23EE
 P 4800 3300
-F 0 "#PWR11" H 4800 3150 50  0001 C CNN
+F 0 "#PWR09" H 4800 3150 50  0001 C CNN
 F 1 "+5V" H 4800 3440 50  0000 C CNN
 F 2 "" H 4800 3300 50  0001 C CNN
@@
 $EndComp
 $Comp
-L +5V #PWR17
+L +5V #PWR010
 U 1 1 595C2423
 P 5400 3900
-F 0 "#PWR17" H 5400 3750 50  0001 C CNN
+F 0 "#PWR010" H 5400 3750 50  0001 C CNN
 F 1 "+5V" V 5500 4050 50  0000 C CNN
 F 2 "" H 5400 3900 50  0001 C CNN
@@
 $EndComp
 $Comp
-L +5V #PWR7
+L +5V #PWR011
 U 1 1 595C271A
 P 4300 3900
-F 0 "#PWR7" H 4300 3750 50  0001 C CNN
+F 0 "#PWR011" H 4300 3750 50  0001 C CNN
 F 1 "+5V" H 4300 4040 50  0000 C CNN
 F 2 "" H 4300 3900 50  0001 C CNN
@@
 $EndComp
 $Comp
-L GND #PWR20
+L GND #PWR012
 U 1 1 595C274F
 P 5750 2700
-F 0 "#PWR20" H 5750 2450 50  0001 C CNN
+F 0 "#PWR012" H 5750 2450 50  0001 C CNN
 F 1 "GND" V 5700 2500 50  0000 C CNN
 F 2 "" H 5750 2700 50  0001 C CNN
@@
 $EndComp
 $Comp
-L VSS #PWR13
+L VSS #PWR013
 U 1 1 595C2784
 P 4900 3800
-F 0 "#PWR13" H 4900 3650 50  0001 C CNN
+F 0 "#PWR013" H 4900 3650 50  0001 C CNN
 F 1 "VSS" V 4900 4000 50  0000 C CNN
 F 2 "" H 4900 3800 50  0001 C CNN
@@
 $EndComp
 $Comp
-L VSS #PWR22
+L VSS #PWR014
 U 1 1 595C27B9
 P 6400 2200
-F 0 "#PWR22" H 6400 2050 50  0001 C CNN
+F 0 "#PWR014" H 6400 2050 50  0001 C CNN
 F 1 "VSS" V 6400 2400 50  0000 C CNN
 F 2 "" H 6400 2200 50  0001 C CNN
@@
 $EndComp
 $Comp
-L GND #PWR24
+L GND #PWR015
 U 1 1 595C27EE
 P 7350 2900
-F 0 "#PWR24" H 7350 2650 50  0001 C CNN
+F 0 "#PWR015" H 7350 2650 50  0001 C CNN
 F 1 "GND" H 7350 2750 50  0000 C CNN
 F 2 "" H 7350 2900 50  0001 C CNN
@@
 $EndComp
 $Comp
-L GND #PWR23
+L GND #PWR016
 U 1 1 595C2A57
 P 6950 3900
-F 0 "#PWR23" H 6950 3650 50  0001 C CNN
+F 0 "#PWR016" H 6950 3650 50  0001 C CNN
 F 1 "GND" V 6900 3700 50  0000 C CNN
 F 2 "" H 6950 3900 50  0001 C CNN
@@
 $EndComp
 $Comp
-L +5V #PWR14
+L +5V #PWR017
 U 1 1 595C2D30
 P 5250 2500
-F 0 "#PWR14" H 5250 2350 50  0001 C CNN
+F 0 "#PWR017" H 5250 2350 50  0001 C CNN
 F 1 "+5V" H 5250 2640 50  0000 C CNN
 F 2 "" H 5250 2500 50  0001 C CNN
@@
 $EndComp
 $Comp
-L GND #PWR15
+L GND #PWR018
 U 1 1 595C2D68
 P 5250 2600
-F 0 "#PWR15" H 5250 2350 50  0001 C CNN
+F 0 "#PWR018" H 5250 2350 50  0001 C CNN
 F 1 "GND" V 5200 2400 50  0000 C CNN
 F 2 "" H 5250 2600 50  0001 C CNN
@@
 $EndComp
 $Comp
-L GND #PWR9
+L GND #PWR019
 U 1 1 595C2DA0
 P 4350 2700
-F 0 "#PWR9" H 4350 2450 50  0001 C CNN
+F 0 "#PWR019" H 4350 2450 50  0001 C CNN
 F 1 "GND" V 4300 2500 50  0000 C CNN
 F 2 "" H 4350 2700 50  0001 C CNN
@@
 $EndComp
 $Comp
-L VSS #PWR8
+L VSS #PWR020
 U 1 1 595C2E3E
 P 4350 2400
-F 0 "#PWR8" H 4350 2250 50  0001 C CNN
+F 0 "#PWR020" H 4350 2250 50  0001 C CNN
 F 1 "VSS" V 4350 2600 50  0000 C CNN
 F 2 "" H 4350 2400 50  0001 C CNN
@@
 BAT-
 $Comp
-L GND #PWR10
+L GND #PWR021
 U 1 1 59A5E3A9
 P 4450 900
-F 0 "#PWR10" H 4450 650 50  0001 C CNN
+F 0 "#PWR021" H 4450 650 50  0001 C CNN
 F 1 "GND" V 4450 700 50  0000 C CNN
 F 2 "" H 4450 900 50  0001 C CNN
@@
 Connection ~ 3900 1250
 $Comp
-L GND #PWR6
+L GND #PWR022
 U 1 1 59A5FF0F
 P 4150 1000
-F 0 "#PWR6" H 4150 750 50  0001 C CNN
+F 0 "#PWR022" H 4150 750 50  0001 C CNN
 F 1 "GND" H 4200 850 50  0000 C CNN
 F 2 "" H 4150 1000 50  0001 C CNN
@@
 	1    0    0    -1
 $EndComp
-Text GLabel 2600 1600 3    60   Input ~ 0
+Text GLabel 2800 1600 3    60   Input ~ 0
 RX_LED
-Text GLabel 2500 1600 3    60   Input ~ 0
+Text GLabel 2700 1600 3    60   Input ~ 0
 TX_LED
 $Comp
@@
 Text GLabel 5900 1750 2    60   Input ~ 0
 RST
-Text GLabel 2800 1600 3    60   Input ~ 0
+Text GLabel 2500 1600 3    60   Input ~ 0
 RST
 Text Label 4550 1150 0    60   ~ 0
 VDD
-Text GLabel 2800 1200 1    60   Input ~ 0
+Text GLabel 2500 1200 1    60   Input ~ 0
 VDD
 $Comp
 L LED D4
 U 1 1 59A60765
-P 2200 1100
-F 0 "D4" H 2200 1200 50  0000 C CNN
-F 1 "LED" H 2200 1000 50  0000 C CNN
-F 2 "Resistors_SMD:R_0603_HandSoldering" H 2200 1100 50  0001 C CNN
-F 3 "" H 2200 1100 50  0001 C CNN
-	1    2200 1100
-	-1   0    0    1
-$EndComp
-$Comp
-L LED D3
-U 1 1 59A607FE
 P 2200 800
-F 0 "D3" H 2200 900 50  0000 C CNN
+F 0 "D4" H 2200 900 50  0000 C CNN
 F 1 "LED" H 2200 700 50  0000 C CNN
 F 2 "Resistors_SMD:R_0603_HandSoldering" H 2200 800 50  0001 C CNN
@@
 	-1   0    0    1
 $EndComp
-Wire Wire Line
-	2350 800  2600 800
-Wire Wire Line
-	2600 800  2600 1200
-Wire Wire Line
-	2350 1100 2500 1100
-Wire Wire Line
-	2500 1100 2500 1200
-$Comp
-L +5V #PWR1
+$Comp
+L LED D3
+U 1 1 59A607FE
+P 3100 800
+F 0 "D3" H 3100 900 50  0000 C CNN
+F 1 "LED" H 3100 700 50  0000 C CNN
+F 2 "Resistors_SMD:R_0603_HandSoldering" H 3100 800 50  0001 C CNN
+F 3 "" H 3100 800 50  0001 C CNN
+	1    3100 800
+	1    0    0    -1
+$EndComp
+Wire Wire Line
+	2350 800  2700 800
+Wire Wire Line
+	2950 800  2800 800
+$Comp
+L +5V #PWR023
 U 1 1 59A6093E
 P 2050 800
-F 0 "#PWR1" H 2050 650 50  0001 C CNN
+F 0 "#PWR023" H 2050 650 50  0001 C CNN
 F 1 "+5V" V 2100 950 50  0000 C CNN
 F 2 "" H 2050 800 50  0001 C CNN
@@
 $EndComp
 $Comp
-L +5V #PWR2
+L +5V #PWR024
 U 1 1 59A609D1
-P 2050 1100
-F 0 "#PWR2" H 2050 950 50  0001 C CNN
-F 1 "+5V" V 2100 1250 50  0000 C CNN
-F 2 "" H 2050 1100 50  0001 C CNN
-F 3 "" H 2050 1100 50  0001 C CNN
-	1    2050 1100
-	0    -1   -1   0
+P 3250 800
+F 0 "#PWR024" H 3250 650 50  0001 C CNN
+F 1 "+5V" V 3300 950 50  0000 C CNN
+F 2 "" H 3250 800 50  0001 C CNN
+F 3 "" H 3250 800 50  0001 C CNN
+	1    3250 800
+	0    1    1    0
 $EndComp
 NoConn ~ 5100 2050
 NoConn ~ 5200 2050
-NoConn ~ 2700 1200
-NoConn ~ 2700 1600
+NoConn ~ 2600 1200
+NoConn ~ 2600 1600
 $Comp
 L TEST_2P J5
@@
 Text GLabel 3350 2450 2    60   Input ~ 0
 TXD
+Wire Wire Line
+	2800 800  2800 1200
+Wire Wire Line
+	2700 800  2700 1200
 $EndSCHEMATC
