File: tp4056_usb_board/tp4056_usb_board.sch (KiCad schematic (older format))
At the start: 22 parts, among them J1 USB_OTG, J2 TP4056, J3 DW01, J4 8205A, J5 TEST_2P, U1 TP4056_BREAKOUT, U2 CP2102N-20P

Commit message: Renaming the TP4056 board files + small fixups
Parts:
- D1, D2, D3, D4: footprint Resistors_SMD:R_0603_HandSoldering -> LEDs:LED_0805
Connections:
- no-connect marks 12 -> 14
Changed lines of the file:
@@
 EESchema Schematic File Version 2
-LIBS:tp4056_breakout-rescue
+LIBS:tp4056_usb_board-rescue
 LIBS:power
 LIBS:device
@@
 LIBS:tp4056_breakout
 LIBS:cp2102n-20p
-LIBS:tp4056_breakout-cache
+LIBS:tp4056_usb_board-cache
 EELAYER 25 0
 EELAYER END
@@
 F 0 "D2" H 5850 3900 50  0000 C CNN
 F 1 "LED" H 5850 3700 50  0000 C CNN
-F 2 "Resistors_SMD:R_0603_HandSoldering" H 5850 3800 50  0001 C CNN
+F 2 "LEDs:LED_0805" H 5850 3800 50  0001 C CNN
 F 3 "" H 5850 3800 50  0001 C CNN
 	1    5850 3800
@@
 F 0 "D1" H 4450 4000 50  0000 C CNN
 F 1 "LED" H 4450 3800 50  0000 C CNN
-F 2 "Resistors_SMD:R_0603_HandSoldering" H 4450 3900 50  0001 C CNN
+F 2 "LEDs:LED_0805" H 4450 3900 50  0001 C CNN
 F 3 "" H 4450 3900 50  0001 C CNN
 	1    4450 3900
@@
 F 0 "D4" H 2200 900 50  0000 C CNN
 F 1 "LED" H 2200 700 50  0000 C CNN
-F 2 "Resistors_SMD:R_0603_HandSoldering" H 2200 800 50  0001 C CNN
+F 2 "LEDs:LED_0805" H 2200 800 50  0001 C CNN
 F 3 "" H 2200 800 50  0001 C CNN
 	1    2200 800
@@
 F 0 "D3" H 3100 900 50  0000 C CNN
 F 1 "LED" H 3100 700 50  0000 C CNN
-F 2 "Resistors_SMD:R_0603_HandSoldering" H 3100 800 50  0001 C CNN
+F 2 "LEDs:LED_0805" H 3100 800 50  0001 C CNN
 F 3 "" H 3100 800 50  0001 C CNN
 	1    3100 800
@@
 Wire Wire Line
 	2700 800  2700 1200
+NoConn ~ 7150 3350
+NoConn ~ 6850 3850
 $EndSCHEMATC

Commit message: Fixing the schematic - adding a jumper (instead of the capacitor) to the TEMP pin
Parts:
- removed C1: C, Capacitors_SMD:C_0603, symbol C
- added JP1: TEMP, footprints:GS2_SMALL, symbol Jumper_NO_Small
Connections:
- net GND: now also JP1.1
- net at J2.1 (P1): now also JP1.2
Changed lines of the file:
@@
-$EndComp
-$Comp
-L C C1
-U 1 1 595C1981
-P 4800 3450
-F 0 "C1" H 4825 3550 50  0000 L CNN
-F 1 "C" H 4825 3350 50  0000 L CNN
-F 2 "Capacitors_SMD:C_0603" H 4838 3300 50  0001 C CNN
-F 3 "" H 4800 3450 50  0001 C CNN
-	1    4800 3450
-	1    0    0    -1
 $EndComp
 $Comp
@@
 L GND #PWR05
 U 1 1 595C1C7D
-P 4900 3700
-F 0 "#PWR05" H 4900 3450 50  0001 C CNN
-F 1 "GND" V 4850 3500 50  0000 C CNN
-F 2 "" H 4900 3700 50  0001 C CNN
-F 3 "" H 4900 3700 50  0001 C CNN
-	1    4900 3700
+P 4550 3700
+F 0 "#PWR05" H 4550 3450 50  0001 C CNN
+F 1 "GND" V 4500 3500 50  0000 C CNN
+F 2 "" H 4550 3700 50  0001 C CNN
+F 3 "" H 4550 3700 50  0001 C CNN
+	1    4550 3700
 	0    1    1    0
 $EndComp
@@
 $Comp
 L +5V #PWR09
-U 1 1 595C23EE
-P 4800 3300
-F 0 "#PWR09" H 4800 3150 50  0001 C CNN
-F 1 "+5V" H 4800 3440 50  0000 C CNN
-F 2 "" H 4800 3300 50  0001 C CNN
-F 3 "" H 4800 3300 50  0001 C CNN
-	1    4800 3300
-	1    0    0    -1
-$EndComp
-$Comp
-L +5V #PWR010
 U 1 1 595C2423
 P 5400 3900
-F 0 "#PWR010" H 5400 3750 50  0001 C CNN
+F 0 "#PWR09" H 5400 3750 50  0001 C CNN
 F 1 "+5V" V 5500 4050 50  0000 C CNN
 F 2 "" H 5400 3900 50  0001 C CNN
@@
 $EndComp
 $Comp
-L +5V #PWR011
+L +5V #PWR010
 U 1 1 595C271A
 P 4300 3900
-F 0 "#PWR011" H 4300 3750 50  0001 C CNN
+F 0 "#PWR010" H 4300 3750 50  0001 C CNN
 F 1 "+5V" H 4300 4040 50  0000 C CNN
 F 2 "" H 4300 3900 50  0001 C CNN
@@
 $EndComp
 $Comp
-L GND #PWR012
+L GND #PWR011
 U 1 1 595C274F
 P 5750 2700
-F 0 "#PWR012" H 5750 2450 50  0001 C CNN
+F 0 "#PWR011" H 5750 2450 50  0001 C CNN
 F 1 "GND" V 5700 2500 50  0000 C CNN
 F 2 "" H 5750 2700 50  0001 C CNN
@@
 $EndComp
 $Comp
-L VSS #PWR013
+L VSS #PWR012
 U 1 1 595C2784
 P 4900 3800
-F 0 "#PWR013" H 4900 3650 50  0001 C CNN
+F 0 "#PWR012" H 4900 3650 50  0001 C CNN
 F 1 "VSS" V 4900 4000 50  0000 C CNN
 F 2 "" H 4900 3800 50  0001 C CNN
@@
 $EndComp
 $Comp
-L VSS #PWR014
+L VSS #PWR013
 U 1 1 595C27B9
 P 6400 2200
-F 0 "#PWR014" H 6400 2050 50  0001 C CNN
+F 0 "#PWR013" H 6400 2050 50  0001 C CNN
 F 1 "VSS" V 6400 2400 50  0000 C CNN
 F 2 "" H 6400 2200 50  0001 C CNN
@@
 $EndComp
 $Comp
-L GND #PWR015
+L GND #PWR014
 U 1 1 595C27EE
 P 7350 2900
-F 0 "#PWR015" H 7350 2650 50  0001 C CNN
+F 0 "#PWR014" H 7350 2650 50  0001 C CNN
 F 1 "GND" H 7350 2750 50  0000 C CNN
 F 2 "" H 7350 2900 50  0001 C CNN
@@
 $EndComp
 $Comp
-L GND #PWR016
+L GND #PWR015
 U 1 1 595C2A57
 P 6950 3900
-F 0 "#PWR016" H 6950 3650 50  0001 C CNN
+F 0 "#PWR015" H 6950 3650 50  0001 C CNN
 F 1 "GND" V 6900 3700 50  0000 C CNN
 F 2 "" H 6950 3900 50  0001 C CNN
@@
 $EndComp
 $Comp
-L +5V #PWR017
+L +5V #PWR016
 U 1 1 595C2D30
 P 5250 2500
-F 0 "#PWR017" H 5250 2350 50  0001 C CNN
+F 0 "#PWR016" H 5250 2350 50  0001 C CNN
 F 1 "+5V" H 5250 2640 50  0000 C CNN
 F 2 "" H 5250 2500 50  0001 C CNN
@@
 $EndComp
 $Comp
-L GND #PWR018
+L GND #PWR017
 U 1 1 595C2D68
 P 5250 2600
-F 0 "#PWR018" H 5250 2350 50  0001 C CNN
+F 0 "#PWR017" H 5250 2350 50  0001 C CNN
 F 1 "GND" V 5200 2400 50  0000 C CNN
 F 2 "" H 5250 2600 50  0001 C CNN
@@
 $EndComp
 $Comp
-L GND #PWR019
+L GND #PWR018
 U 1 1 595C2DA0
 P 4350 2700
-F 0 "#PWR019" H 4350 2450 50  0001 C CNN
+F 0 "#PWR018" H 4350 2450 50  0001 C CNN
 F 1 "GND" V 4300 2500 50  0000 C CNN
 F 2 "" H 4350 2700 50  0001 C CNN
@@
 $EndComp
 $Comp
-L VSS #PWR020
+L VSS #PWR019
 U 1 1 595C2E3E
 P 4350 2400
-F 0 "#PWR020" H 4350 2250 50  0001 C CNN
+F 0 "#PWR019" H 4350 2250 50  0001 C CNN
 F 1 "VSS" V 4350 2600 50  0000 C CNN
 F 2 "" H 4350 2400 50  0001 C CNN
@@
 BAT-
 $Comp
-L GND #PWR021
+L GND #PWR020
 U 1 1 59A5E3A9
 P 4450 900
-F 0 "#PWR021" H 4450 650 50  0001 C CNN
+F 0 "#PWR020" H 4450 650 50  0001 C CNN
 F 1 "GND" V 4450 700 50  0000 C CNN
 F 2 "" H 4450 900 50  0001 C CNN
@@
 $EndComp
 Wire Wire Line
-	4800 3600 4900 3600
-Wire Wire Line
 	5400 3600 5500 3600
 Wire Wire Line
@@
 Connection ~ 3900 1250
 $Comp
-L GND #PWR022
+L GND #PWR021
 U 1 1 59A5FF0F
 P 4150 1000
-F 0 "#PWR022" H 4150 750 50  0001 C CNN
+F 0 "#PWR021" H 4150 750 50  0001 C CNN
 F 1 "GND" H 4200 850 50  0000 C CNN
 F 2 "" H 4150 1000 50  0001 C CNN
@@
 	2950 800  2800 800
 $Comp
-L +5V #PWR023
+L +5V #PWR022
 U 1 1 59A6093E
 P 2050 800
-F 0 "#PWR023" H 2050 650 50  0001 C CNN
+F 0 "#PWR022" H 2050 650 50  0001 C CNN
 F 1 "+5V" V 2100 950 50  0000 C CNN
 F 2 "" H 2050 800 50  0001 C CNN
@@
 $EndComp
 $Comp
-L +5V #PWR024
+L +5V #PWR023
 U 1 1 59A609D1
 P 3250 800
-F 0 "#PWR024" H 3250 650 50  0001 C CNN
+F 0 "#PWR023" H 3250 650 50  0001 C CNN
 F 1 "+5V" V 3300 950 50  0000 C CNN
 F 2 "" H 3250 800 50  0001 C CNN
@@
 NoConn ~ 7150 3350
 NoConn ~ 6850 3850
+$Comp
+L Jumper_NO_Small JP1
+U 1 1 5AE60494
+P 4800 3600
+F 0 "JP1" H 4800 3680 50  0000 C CNN
+F 1 "TEMP" H 4810 3540 50  0000 C CNN
+F 2 "footprints:GS2_SMALL" H 4800 3600 50  0001 C CNN
+F 3 "" H 4800 3600 50  0001 C CNN
+	1    4800 3600
+	1    0    0    -1
+$EndComp
+Wire Wire Line
+	4550 3700 4900 3700
+Wire Wire Line
+	4600 3700 4600 3600
+Wire Wire Line
+	4600 3600 4700 3600
+Connection ~ 4600 3700
 $EndSCHEMATC

Commit message: TP4056 board - changing current set resistor FP to 1206 (better change to 0805 in the next rev?)
Parts:
- R2: footprint Resistors_SMD:R_0603 -> Resistors_SMD:R_1206
Changed lines of the file:
@@
 F 0 "R2" V 5580 3450 50  0000 C CNN
 F 1 "R" V 5500 3450 50  0000 C CNN
-F 2 "Resistors_SMD:R_0603" V 5430 3450 50  0001 C CNN
+F 2 "Resistors_SMD:R_1206" V 5430 3450 50  0001 C CNN
 F 3 "" H 5500 3450 50  0001 C CNN
 	1    5500 3450
