File: audio_buffer/audio_buffer.kicad_pcb (KiCad board)
At the start: 2 copper layers, 13.2 x 10.7 mm, 9 parts, among them P1 INPUT_CONN, P2 OUTPUT_CONN, U1 MIC5219-3.3BM5, U2 NC7WZ16

Commit message: Added version information
Other:
- board text added: "v1.1"
Changed lines of the file:
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@@
-(kicad_pcb (version 4) (host pcbnew 4.0.6)
+(kicad_pcb (version 4) (host pcbnew 4.0.7)
   (general
     (links 17)
-    (no_connects 7)
-    (area 121.514286 90.615 141.979048 105.831428)
+    (no_connects 0)
+    (area 125.400999 92.380999 138.759001 103.199001)
     (thickness 1.6)
-    (drawings 4)
+    (drawings 5)
     (tracks 47)
     (zones 0)
@@
   )
   (setup
-    (last_trace_width 0.5)
+    (last_trace_width 0.25)
     (user_trace_width 0.4)
     (user_trace_width 0.5)
@@
     )
   )
+  (gr_text v1.1 (at 132 101.6) (layer F.SilkS)
+    (effects (font (size 1 1) (thickness 0.15)))
+  )
   (gr_line (start 125.476 103.124) (end 125.476 92.456) (layer Edge.Cuts) (width 0.15))

Commit message: Fixed pin header 3D model offsets
Parts:
- P1, P2: moved to B.Cu
- turned P2 to 0 degrees
- turned P1 to 0 degrees
Changed lines of the file:
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@@
     (add_net VCC)
   )
-  (module Pin_Headers:Pin_Header_Straight_1x03_Pitch2.54mm (layer F.Cu)
-    (at 137.16 101.6 180)
+  (module Pin_Headers:Pin_Header_Straight_1x03_Pitch2.54mm (layer B.Cu)
+    (at 137.16 101.6)
     (descr "Through hole straight pin header, 1x03, 2.54mm pitch, single row")
     (tags "Through hole pin header THT 1x03 2.54mm single row")
-    (fp_text reference P1 (at 0 -2.39 180) (layer F.SilkS) hide
-      (effects (font (size 1 1) (thickness 0.15)))
+    (fp_text reference P1 (at 0 2.39) (layer B.SilkS) hide
+      (effects (font (size 1 1) (thickness 0.15)) (justify mirror))
     )
-    (fp_text value INPUT_CONN (at 0 7.47 180) (layer F.Fab) hide
-      (effects (font (size 1 1) (thickness 0.15)))
+    (fp_text value INPUT_CONN (at 0 -7.47) (layer B.Fab) hide
+      (effects (font (size 1 1) (thickness 0.15)) (justify mirror))
     )
-    (fp_line (start -1.27 -1.27) (end -1.27 6.35) (layer F.Fab) (width 0.1))
-    (fp_line (start -1.27 6.35) (end 1.27 6.35) (layer F.Fab) (width 0.1))
-    (fp_line (start 1.27 6.35) (end 1.27 -1.27) (layer F.Fab) (width 0.1))
-    (fp_line (start 1.27 -1.27) (end -1.27 -1.27) (layer F.Fab) (width 0.1))
-    (fp_line (start -1.39 1.27) (end -1.39 6.47) (layer F.SilkS) (width 0.12))
-    (fp_line (start -1.39 6.47) (end 1.39 6.47) (layer F.SilkS) (width 0.12))
-    (fp_line (start 1.39 6.47) (end 1.39 1.27) (layer F.SilkS) (width 0.12))
-    (fp_line (start 1.39 1.27) (end -1.39 1.27) (layer F.SilkS) (width 0.12))
-    (fp_line (start -1.39 0) (end -1.39 -1.39) (layer F.SilkS) (width 0.12))
-    (fp_line (start -1.39 -1.39) (end 0 -1.39) (layer F.SilkS) (width 0.12))
-    (fp_line (start -1.6 -1.6) (end -1.6 6.6) (layer F.CrtYd) (width 0.05))
-    (fp_line (start -1.6 6.6) (end 1.6 6.6) (layer F.CrtYd) (width 0.05))
-    (fp_line (start 1.6 6.6) (end 1.6 -1.6) (layer F.CrtYd) (width 0.05))
-    (fp_line (start 1.6 -1.6) (end -1.6 -1.6) (layer F.CrtYd) (width 0.05))
-    (pad 1 thru_hole rect (at 0 0 180) (size 1.7 1.7) (drill 1) (layers *.Cu *.Mask)
+    (fp_line (start -1.27 1.27) (end -1.27 -6.35) (layer B.Fab) (width 0.1))
+    (fp_line (start -1.27 -6.35) (end 1.27 -6.35) (layer B.Fab) (width 0.1))
+    (fp_line (start 1.27 -6.35) (end 1.27 1.27) (layer B.Fab) (width 0.1))
+    (fp_line (start 1.27 1.27) (end -1.27 1.27) (layer B.Fab) (width 0.1))
+    (fp_line (start -1.39 -1.27) (end -1.39 -6.47) (layer B.SilkS) (width 0.12))
+    (fp_line (start -1.39 -6.47) (end 1.39 -6.47) (layer B.SilkS) (width 0.12))
+    (fp_line (start 1.39 -6.47) (end 1.39 -1.27) (layer B.SilkS) (width 0.12))
+    (fp_line (start 1.39 -1.27) (end -1.39 -1.27) (layer B.SilkS) (width 0.12))
+    (fp_line (start -1.39 0) (end -1.39 1.39) (layer B.SilkS) (width 0.12))
+    (fp_line (start -1.39 1.39) (end 0 1.39) (layer B.SilkS) (width 0.12))
+    (fp_line (start -1.6 1.6) (end -1.6 -6.6) (layer B.CrtYd) (width 0.05))
+    (fp_line (start -1.6 -6.6) (end 1.6 -6.6) (layer B.CrtYd) (width 0.05))
+    (fp_line (start 1.6 -6.6) (end 1.6 1.6) (layer B.CrtYd) (width 0.05))
+    (fp_line (start 1.6 1.6) (end -1.6 1.6) (layer B.CrtYd) (width 0.05))
+    (pad 1 thru_hole rect (at 0 0) (size 1.7 1.7) (drill 1) (layers *.Cu *.Mask)
       (net 2 "Net-(P1-Pad1)"))
-    (pad 2 thru_hole oval (at 0 2.54 180) (size 1.7 1.7) (drill 1) (layers *.Cu *.Mask)
+    (pad 2 thru_hole oval (at 0 -2.54) (size 1.7 1.7) (drill 1) (layers *.Cu *.Mask)
       (net 9 VCC))
-    (pad 3 thru_hole oval (at 0 5.08 180) (size 1.7 1.7) (drill 1) (layers *.Cu *.Mask)
+    (pad 3 thru_hole oval (at 0 -5.08) (size 1.7 1.7) (drill 1) (layers *.Cu *.Mask)
       (net 3 "Net-(P1-Pad3)"))
     (model Pin_Headers.3dshapes/Pin_Header_Straight_1x03_Pitch2.54mm.wrl
-      (at (xyz 0 -0.1 0))
+      (at (xyz 0 0 0))
       (scale (xyz 1 1 1))
-      (rotate (xyz 0 0 90))
+      (rotate (xyz 0 0 0))
     )
   )
-  (module Pin_Headers:Pin_Header_Straight_1x04_Pitch2.54mm (layer F.Cu)
-    (at 127 101.6 180)
+  (module Pin_Headers:Pin_Header_Straight_1x04_Pitch2.54mm (layer B.Cu)
+    (at 126.9746 101.6)
     (descr "Through hole straight pin header, 1x04, 2.54mm pitch, single row")
     (tags "Through hole pin header THT 1x04 2.54mm single row")
-    (fp_text reference P2 (at 0 -2.39 180) (layer F.SilkS) hide
-      (effects (font (size 1 1) (thickness 0.15)))
+    (fp_text reference P2 (at 0 2.39) (layer B.SilkS) hide
+      (effects (font (size 1 1) (thickness 0.15)) (justify mirror))
     )
-    (fp_text value OUTPUT_CONN (at 0 10.01 180) (layer F.Fab) hide
-      (effects (font (size 1 1) (thickness 0.15)))
+    (fp_text value OUTPUT_CONN (at 0 -10.01) (layer B.Fab) hide
+      (effects (font (size 1 1) (thickness 0.15)) (justify mirror))
     )
-    (fp_line (start -1.27 -1.27) (end -1.27 8.89) (layer F.Fab) (width 0.1))
-    (fp_line (start -1.27 8.89) (end 1.27 8.89) (layer F.Fab) (width 0.1))
-    (fp_line (start 1.27 8.89) (end 1.27 -1.27) (layer F.Fab) (width 0.1))
-    (fp_line (start 1.27 -1.27) (end -1.27 -1.27) (layer F.Fab) (width 0.1))
-    (fp_line (start -1.39 1.27) (end -1.39 9.01) (layer F.SilkS) (width 0.12))
-    (fp_line (start -1.39 9.01) (end 1.39 9.01) (layer F.SilkS) (width 0.12))
-    (fp_line (start 1.39 9.01) (end 1.39 1.27) (layer F.SilkS) (width 0.12))
-    (fp_line (start 1.39 1.27) (end -1.39 1.27) (layer F.SilkS) (width 0.12))
-    (fp_line (start -1.39 0) (end -1.39 -1.39) (layer F.SilkS) (width 0.12))
-    (fp_line (start -1.39 -1.39) (end 0 -1.39) (layer F.SilkS) (width 0.12))
-    (fp_line (start -1.6 -1.6) (end -1.6 9.2) (layer F.CrtYd) (width 0.05))
-    (fp_line (start -1.6 9.2) (end 1.6 9.2) (layer F.CrtYd) (width 0.05))
-    (fp_line (start 1.6 9.2) (end 1.6 -1.6) (layer F.CrtYd) (width 0.05))
-    (fp_line (start 1.6 -1.6) (end -1.6 -1.6) (layer F.CrtYd) (width 0.05))
-    (pad 1 thru_hole rect (at 0 0 180) (size 1.7 1.7) (drill 1) (layers *.Cu *.Mask)
+    (fp_line (start -1.27 1.27) (end -1.27 -8.89) (layer B.Fab) (width 0.1))
+    (fp_line (start -1.27 -8.89) (end 1.27 -8.89) (layer B.Fab) (width 0.1))
+    (fp_line (start 1.27 -8.89) (end 1.27 1.27) (layer B.Fab) (width 0.1))
+    (fp_line (start 1.27 1.27) (end -1.27 1.27) (layer B.Fab) (width 0.1))
+    (fp_line (start -1.39 -1.27) (end -1.39 -9.01) (layer B.SilkS) (width 0.12))
+    (fp_line (start -1.39 -9.01) (end 1.39 -9.01) (layer B.SilkS) (width 0.12))
+    (fp_line (start 1.39 -9.01) (end 1.39 -1.27) (layer B.SilkS) (width 0.12))
+    (fp_line (start 1.39 -1.27) (end -1.39 -1.27) (layer B.SilkS) (width 0.12))
+    (fp_line (start -1.39 0) (end -1.39 1.39) (layer B.SilkS) (width 0.12))
+    (fp_line (start -1.39 1.39) (end 0 1.39) (layer B.SilkS) (width 0.12))
+    (fp_line (start -1.6 1.6) (end -1.6 -9.2) (layer B.CrtYd) (width 0.05))
+    (fp_line (start -1.6 -9.2) (end 1.6 -9.2) (layer B.CrtYd) (width 0.05))
+    (fp_line (start 1.6 -9.2) (end 1.6 1.6) (layer B.CrtYd) (width 0.05))
+    (fp_line (start 1.6 1.6) (end -1.6 1.6) (layer B.CrtYd) (width 0.05))
+    (pad 1 thru_hole rect (at 0 0) (size 1.7 1.7) (drill 1) (layers *.Cu *.Mask)
       (net 4 "Net-(P2-Pad1)"))
-    (pad 2 thru_hole oval (at 0 2.54 180) (size 1.7 1.7) (drill 1) (layers *.Cu *.Mask)
+    (pad 2 thru_hole oval (at 0 -2.54) (size 1.7 1.7) (drill 1) (layers *.Cu *.Mask)
       (net 1 GND))
-    (pad 3 thru_hole oval (at 0 5.08 180) (size 1.7 1.7) (drill 1) (layers *.Cu *.Mask)
+    (pad 3 thru_hole oval (at 0 -5.08) (size 1.7 1.7) (drill 1) (layers *.Cu *.Mask)
       (net 5 "Net-(P2-Pad3)"))
-    (pad 4 thru_hole oval (at 0 7.62 180) (size 1.7 1.7) (drill 1) (layers *.Cu *.Mask)
+    (pad 4 thru_hole oval (at 0 -7.62) (size 1.7 1.7) (drill 1) (layers *.Cu *.Mask)
       (net 6 "Net-(P2-Pad4)"))
     (model Pin_Headers.3dshapes/Pin_Header_Straight_1x04_Pitch2.54mm.wrl
-      (at (xyz 0 -0.15 0))
+      (at (xyz 0 0 0))
       (scale (xyz 1 1 1))
-      (rotate (xyz 0 0 90))
+      (rotate (xyz 0 0 0))
     )
   )
