File: esp12_1button_6leds/esp12_1button_6leds.kicad_pcb (KiCad board)
At the start: 2 copper layers, 16 x 24 mm, 15 parts, among them SW1 SW_Push, U1 ESP-12E

Commit message: Added some stub traces to fix non-connects
Routing:
- net Net-(U1-Pad7): track 0.00 -> 1.00 mm
- net Net-(U1-Pad6): track 0.00 -> 1.00 mm
- net Net-(U1-Pad5): track 0.00 -> 1.00 mm
- net Net-(U1-Pad4): track 0.00 -> 1.00 mm
- net Net-(U1-Pad22): track 0.00 -> 1.00 mm
- net Net-(U1-Pad21): track 0.00 -> 1.00 mm
- net Net-(U1-Pad20): track 0.00 -> 1.00 mm
- net Net-(U1-Pad2): track 0.00 -> 1.00 mm
- net Net-(U1-Pad19): track 0.00 -> 1.00 mm
- net Net-(U1-Pad18): track 0.00 -> 1.00 mm
- net Net-(U1-Pad17): track 0.00 -> 1.00 mm
- net Net-(U1-Pad16): track 0.00 -> 1.00 mm
- net Net-(U1-Pad1): track 0.00 -> 1.00 mm
- net Net-(R1-Pad2): track 32.3 -> 33.3 mm
- net GND: track 44.4 -> 45.4 mm
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Other:
- board text added: "ESP12-LED mod for ZeroPhone v1.0, by CRImier"
Changed lines of the file:
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@@
-(kicad_pcb (version 4) (host pcbnew 4.0.6)
+(kicad_pcb (version 4) (host pcbnew 4.0.7)
   (general
     (links 40)
@@
     (area 139.425 90.2972 158.025 117.7036)
     (thickness 1.6)
-    (drawings 1)
-    (tracks 101)
+    (drawings 2)
+    (tracks 117)
     (zones 0)
     (modules 15)
@@
     )
   )
+  (gr_text "ESP12-LED mod\nfor ZeroPhone\nv1.0, by CRImier" (at 148.5 106) (layer F.SilkS)
+    (effects (font (size 0.9 0.9) (thickness 0.18)))
+  )
   (gr_text "1xSW, 6xLED" (at 148.5 98.1 180) (layer B.SilkS)
     (effects (font (size 1.5 1.5) (thickness 0.3)) (justify mirror))
   )
+  (segment (start 140.5011 101.5036) (end 141.5011 101.5036) (width 0.25) (layer B.Cu) (net 1))
+  (segment (start 140.5011 103.5036) (end 141.5011 103.5036) (width 0.25) (layer B.Cu) (net 2))
+  (segment (start 140.5011 107.5036) (end 141.5011 107.5036) (width 0.25) (layer B.Cu) (net 3))
+  (segment (start 140.5011 109.5036) (end 141.5011 109.5036) (width 0.25) (layer B.Cu) (net 4))
+  (segment (start 140.5011 111.5036) (end 141.5011 111.5036) (width 0.25) (layer B.Cu) (net 5))
+  (segment (start 140.5011 113.5036) (end 141.5011 113.5036) (width 0.25) (layer B.Cu) (net 6))
+  (segment (start 156.5011 113.5036) (end 155.5011 113.5036) (width 0.25) (layer B.Cu) (net 7))
+  (segment (start 156.5011 111.5036) (end 155.5011 111.5036) (width 0.25) (layer B.Cu) (net 8))
+  (segment (start 156.5011 109.5036) (end 155.5011 109.5036) (width 0.25) (layer B.Cu) (net 9))
+  (segment (start 156.5011 107.5036) (end 155.5011 107.5036) (width 0.25) (layer B.Cu) (net 10))
+  (segment (start 156.5011 105.5036) (end 155.5011 105.5036) (width 0.25) (layer B.Cu) (net 11))
+  (segment (start 156.5011 103.5036) (end 155.5011 103.5036) (width 0.25) (layer B.Cu) (net 12))
+  (segment (start 156.5011 101.5036) (end 155.5011 101.5036) (width 0.25) (layer B.Cu) (net 13))
   (segment (start 145.1 100) (end 145.1 112) (width 0.25) (layer F.Cu) (net 14))
   (segment (start 142 95) (end 142 96.9) (width 0.25) (layer F.Cu) (net 14))
@@
   (segment (start 153.5011 97.6989) (end 155.2 96) (width 0.25) (layer B.Cu) (net 25))
   (segment (start 155.2 96) (end 155.25 96) (width 0.25) (layer B.Cu) (net 25))
+  (segment (start 140.5011 115.5036) (end 141.5011 115.5036) (width 0.25) (layer B.Cu) (net 26))
   (segment (start 142.75 115.0047) (end 143.3547 115.0047) (width 0.25) (layer F.Cu) (net 26))
   (segment (start 143.3547 115.0047) (end 143.4 115.05) (width 0.25) (layer F.Cu) (net 26))
   (segment (start 141.5011 115.5036) (end 142.2511 115.5036) (width 0.25) (layer F.Cu) (net 26))
   (segment (start 142.2511 115.5036) (end 142.75 115.0047) (width 0.25) (layer F.Cu) (net 26))
+  (segment (start 140.5011 105.5036) (end 141.5011 105.5036) (width 0.25) (layer B.Cu) (net 27))
   (segment (start 143.4 100.2) (end 143.4 105.5) (width 0.25) (layer F.Cu) (net 27))
   (segment (start 141.2 94.4) (end 141.2 98) (width 0.25) (layer F.Cu) (net 27))
@@
   (segment (start 143.3964 105.5036) (end 143.4 105.5) (width 0.25) (layer F.Cu) (net 27))
   (segment (start 143.4 112) (end 143.4 112.85) (width 0.25) (layer F.Cu) (net 27))
+  (segment (start 156.5011 115.5036) (end 155.5011 115.5036) (width 0.25) (layer B.Cu) (net 28))
   (segment (start 154.3 111.3) (end 154.3 115.0525) (width 0.25) (layer B.Cu) (net 28))
   (segment (start 154.3 115.0525) (end 154.7511 115.5036) (width 0.25) (layer B.Cu) (net 28))
