File: esp12_template/esp12_template.kicad_pcb (KiCad board)
At the start: 2 copper layers, 16 x 24 mm, 1 part, among them U1 ESP-12E

Commit message: Fixing non-connects in ESP12 mod board template
Routing:
- net Net-(U1-Pad7): track 0.00 -> 1.00 mm
- net Net-(U1-Pad6): track 0.00 -> 1.00 mm
- net Net-(U1-Pad5): track 0.00 -> 1.00 mm
- net Net-(U1-Pad4): track 0.00 -> 1.00 mm
- net Net-(U1-Pad3): track 0.00 -> 1.00 mm
- net Net-(U1-Pad22): track 0.00 -> 1.00 mm
- net Net-(U1-Pad21): track 0.00 -> 1.00 mm
- net Net-(U1-Pad20): track 0.00 -> 1.00 mm
- net Net-(U1-Pad2): track 0.00 -> 1.00 mm
- net Net-(U1-Pad19): track 0.00 -> 1.00 mm
- net Net-(U1-Pad18): track 0.00 -> 1.00 mm
- net Net-(U1-Pad17): track 0.00 -> 1.00 mm
- net Net-(U1-Pad16): track 0.00 -> 1.00 mm
- net Net-(U1-Pad1): track 0.00 -> 1.00 mm
- net GND: track 0.00 -> 1.00 mm
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Changed lines of the file:
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@@
-(kicad_pcb (version 4) (host pcbnew 4.0.6)
+(kicad_pcb (version 4) (host pcbnew 4.0.7)
   (general
     (links 16)
@@
     (thickness 1.6)
     (drawings 0)
-    (tracks 0)
+    (tracks 16)
     (zones 0)
     (modules 1)
@@
       (net 14 "Net-(U1-Pad22)"))
   )
+  (segment (start 140.5011 101.5036) (end 141.5011 101.5036) (width 0.25) (layer F.Cu) (net 1))
+  (segment (start 140.5011 103.5036) (end 141.5011 103.5036) (width 0.25) (layer F.Cu) (net 2))
+  (segment (start 140.5011 105.5036) (end 141.5011 105.5036) (width 0.25) (layer F.Cu) (net 3))
+  (segment (start 140.5011 107.5036) (end 141.5011 107.5036) (width 0.25) (layer F.Cu) (net 4))
+  (segment (start 140.5011 109.5036) (end 141.5011 109.5036) (width 0.25) (layer F.Cu) (net 5))
+  (segment (start 140.5011 111.5036) (end 141.5011 111.5036) (width 0.25) (layer F.Cu) (net 6))
+  (segment (start 141.5011 113.5036) (end 140.5011 113.5036) (width 0.25) (layer F.Cu) (net 7))
+  (segment (start 156.5011 113.5036) (end 155.5011 113.5036) (width 0.25) (layer F.Cu) (net 8))
+  (segment (start 156.5011 111.5036) (end 155.5011 111.5036) (width 0.25) (layer F.Cu) (net 9))
+  (segment (start 156.5011 109.5036) (end 155.5011 109.5036) (width 0.25) (layer F.Cu) (net 10))
+  (segment (start 155.5011 107.5036) (end 156.5011 107.5036) (width 0.25) (layer F.Cu) (net 11))
+  (segment (start 156.5011 105.5036) (end 155.5011 105.5036) (width 0.25) (layer F.Cu) (net 12))
+  (segment (start 155.5011 103.5036) (end 156.5011 103.5036) (width 0.25) (layer F.Cu) (net 13))
+  (segment (start 156.5011 101.5036) (end 155.5011 101.5036) (width 0.25) (layer F.Cu) (net 14))
+  (segment (start 141.5011 115.5036) (end 140.5011 115.5036) (width 0.25) (layer F.Cu) (net 15))
+  (segment (start 156.5011 115.5036) (end 155.5011 115.5036) (width 0.25) (layer F.Cu) (net 16))
 )
