File: enc28j60_breakout_adapter/enc28j60_breakout_adapter.kicad_pcb (KiCad board)
At the start: 2 copper layers, 27.3 x 21.6 mm, 4 parts, among them J1 CONN_02X05, J2 CONN_01X07, J3 INT

Commit message: Adjusted silkscreen
Other:
- board text added: "ENC28J60 breakout v1.0"
- board text added: "by CRImier, v1.0"
- board text removed: "modprobe enc28j60"
- board text removed: "v1.0"
Changed lines of the file:
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@@
-(kicad_pcb (version 4) (host pcbnew 4.0.6)
+(kicad_pcb (version 4) (host pcbnew 4.0.7)
   (general
     (links 10)
-    (no_connects 1)
+    (no_connects 0)
     (area 145.339999 91.999999 172.795001 113.740001)
     (thickness 1.6)
@@
     (pad_to_mask_clearance 0.2)
     (aux_axis_origin 172.72 92.075)
-    (visible_elements FFFFFF7F)
+    (visible_elements 7FFFFFFF)
     (pcbplotparams
       (layerselection 0x010f0_80000001)
@@
     (effects (font (size 1 1) (thickness 0.25)) (justify mirror))
   )
-  (gr_text "modprobe enc28j60" (at 155.575 93.345) (layer F.SilkS)
+  (gr_text "ENC28J60 breakout v1.0" (at 155.5 94) (layer F.SilkS)
     (effects (font (size 1 1) (thickness 0.25)))
   )
-  (gr_text v1.0 (at 148.59 93.98) (layer B.SilkS)
+  (gr_text "by CRImier, v1.0" (at 153 93.98) (layer B.SilkS)
     (effects (font (size 1 1) (thickness 0.25)) (justify mirror))
   )
