File: level_shifter_adapter/level_shifter_adapter.sch (KiCad schematic (older format))
At the start: 45 parts, among them J1 Conn_01x12, J2 Conn_01x12, Q1 BC847, Q2 IRLML6401, Q3 BC847, Q4 IRLML6401, Q5 BC847, U1 GTL2003, U2 MCP1703A-1802_SOT223, U3 ATTINY45-20SU

Commit message: Level shifter finished and fixed - swapping the MCP for 1117
Parts:
- removed U2: MCP1703A-1802_SOT223, TO_SOT_Packages_SMD:SOT-223-3_TabPin2, symbol MCP1703A-1802_SOT223
- added U2: AP1117-18, TO_SOT_Packages_SMD:SOT-223-3Lead_TabPin2, symbol AP1117-18
Connections:
- net +1V8: now also U2.2 (VO)
- net GND: now also U2.1 (GND)
- net HVCC: now also U2.3 (VI)
Changed lines of the file:
@@
 $EndComp
 $Comp
-L GND #PWR01
+L GND #PWR3
 U 1 1 5AE81C15
 P 1300 1950
-F 0 "#PWR01" H 1300 1700 50  0001 C CNN
+F 0 "#PWR3" H 1300 1700 50  0001 C CNN
 F 1 "GND" V 1300 1750 50  0000 C CNN
 F 2 "" H 1300 1950 50  0001 C CNN
@@
 $EndComp
 $Comp
-L GND #PWR02
+L GND #PWR4
 U 1 1 5AE81C5C
 P 1300 2450
-F 0 "#PWR02" H 1300 2200 50  0001 C CNN
+F 0 "#PWR4" H 1300 2200 50  0001 C CNN
 F 1 "GND" V 1300 2250 50  0000 C CNN
 F 2 "" H 1300 2450 50  0001 C CNN
@@
 $EndComp
 $Comp
-L +5V #PWR03
+L +5V #PWR5
 U 1 1 5AE81C6F
 P 1300 2550
-F 0 "#PWR03" H 1300 2400 50  0001 C CNN
+F 0 "#PWR5" H 1300 2400 50  0001 C CNN
 F 1 "+5V" V 1400 2600 50  0000 C CNN
 F 2 "" H 1300 2550 50  0001 C CNN
@@
 L7
 $Comp
-L GND #PWR04
+L GND #PWR13
 U 1 1 5AE824DD
 P 2550 1550
-F 0 "#PWR04" H 2550 1300 50  0001 C CNN
+F 0 "#PWR13" H 2550 1300 50  0001 C CNN
 F 1 "GND" V 2550 1350 50  0000 C CNN
 F 2 "" H 2550 1550 50  0001 C CNN
@@
 $EndComp
 $Comp
-L GND #PWR05
+L GND #PWR18
 U 1 1 5AE829DB
 P 4750 2050
-F 0 "#PWR05" H 4750 1800 50  0001 C CNN
+F 0 "#PWR18" H 4750 1800 50  0001 C CNN
 F 1 "GND" V 4750 1850 50  0000 C CNN
 F 2 "" H 4750 2050 50  0001 C CNN
@@
 $EndComp
 $Comp
-L GND #PWR06
+L GND #PWR19
 U 1 1 5AE829E1
 P 4750 2550
-F 0 "#PWR06" H 4750 2300 50  0001 C CNN
+F 0 "#PWR19" H 4750 2300 50  0001 C CNN
 F 1 "GND" V 4750 2350 50  0000 C CNN
 F 2 "" H 4750 2550 50  0001 C CNN
@@
 $EndComp
 $Comp
-L +5V #PWR07
+L +5V #PWR20
 U 1 1 5AE829E7
 P 4750 2650
-F 0 "#PWR07" H 4750 2500 50  0001 C CNN
+F 0 "#PWR20" H 4750 2500 50  0001 C CNN
 F 1 "+5V" V 4850 2700 50  0000 C CNN
 F 2 "" H 4750 2650 50  0001 C CNN
@@
 $EndComp
 $Comp
-L GND #PWR08
+L GND #PWR15
 U 1 1 5AE839EF
 P 3850 1550
-F 0 "#PWR08" H 3850 1300 50  0001 C CNN
+F 0 "#PWR15" H 3850 1300 50  0001 C CNN
 F 1 "GND" V 3850 1350 50  0000 C CNN
 F 2 "" H 3850 1550 50  0001 C CNN
@@
 HVCC
 $Comp
-L MCP1703A-1802_SOT223 U2
-U 1 1 5AE8504F
-P 1450 5100
-F 0 "U2" H 1300 5225 50  0000 C CNN
-F 1 "MCP1703A-1802_SOT223" H 500 4550 50  0000 L CNN
-F 2 "TO_SOT_Packages_SMD:SOT-223-3_TabPin2" H 1450 5300 50  0001 C CNN
-F 3 "" H 1450 5050 50  0001 C CNN
-	1    1450 5100
-	1    0    0    -1
-$EndComp
-$Comp
-L +1V8 #PWR09
+L +1V8 #PWR8
 U 1 1 5AE85CCC
 P 1900 5100
-F 0 "#PWR09" H 1900 4950 50  0001 C CNN
+F 0 "#PWR8" H 1900 4950 50  0001 C CNN
 F 1 "+1V8" H 1900 5240 50  0000 C CNN
 F 2 "" H 1900 5100 50  0001 C CNN
@@
 $EndComp
 $Comp
-L GND #PWR010
+L GND #PWR6
 U 1 1 5AE85DA0
 P 1450 5400
-F 0 "#PWR010" H 1450 5150 50  0001 C CNN
+F 0 "#PWR6" H 1450 5150 50  0001 C CNN
 F 1 "GND" H 1450 5250 50  0000 C CNN
 F 2 "" H 1450 5400 50  0001 C CNN
@@
 	1800 5800 1750 5800
 $Comp
-L GND #PWR011
+L GND #PWR12
 U 1 1 5AE87AC6
 P 2400 5900
-F 0 "#PWR011" H 2400 5650 50  0001 C CNN
+F 0 "#PWR12" H 2400 5650 50  0001 C CNN
 F 1 "GND" H 2400 5750 50  0000 C CNN
 F 2 "" H 2400 5900 50  0001 C CNN
@@
 $EndComp
 $Comp
-L +5V #PWR012
+L +5V #PWR1
 U 1 1 5AE88ACB
 P 1050 6300
-F 0 "#PWR012" H 1050 6150 50  0001 C CNN
+F 0 "#PWR1" H 1050 6150 50  0001 C CNN
 F 1 "+5V" V 1150 6350 50  0000 C CNN
 F 2 "" H 1050 6300 50  0001 C CNN
@@
 	1350 6900 1400 6900
 $Comp
-L GND #PWR013
+L GND #PWR7
 U 1 1 5AE88C81
 P 1700 7100
-F 0 "#PWR013" H 1700 6850 50  0001 C CNN
+F 0 "#PWR7" H 1700 6850 50  0001 C CNN
 F 1 "GND" H 1700 6950 50  0000 C CNN
 F 2 "" H 1700 7100 50  0001 C CNN
@@
 $EndComp
 $Comp
-L GND #PWR014
+L GND #PWR23
 U 1 1 5AE89E9D
 P 5900 7050
-F 0 "#PWR014" H 5900 6800 50  0001 C CNN
+F 0 "#PWR23" H 5900 6800 50  0001 C CNN
 F 1 "GND" V 5900 6850 50  0000 C CNN
 F 2 "" H 5900 7050 50  0001 C CNN
@@
 5V_HV_EN
 $Comp
-L +5V #PWR015
+L +5V #PWR11
 U 1 1 5AE8C52D
 P 2200 7600
-F 0 "#PWR015" H 2200 7450 50  0001 C CNN
+F 0 "#PWR11" H 2200 7450 50  0001 C CNN
 F 1 "+5V" V 2200 7800 50  0000 C CNN
 F 2 "" H 2200 7600 50  0001 C CNN
@@
 $EndComp
 $Comp
-L VCC #PWR016
+L VCC #PWR22
 U 1 1 5AE8F999
 P 5900 6550
-F 0 "#PWR016" H 5900 6400 50  0001 C CNN
+F 0 "#PWR22" H 5900 6400 50  0001 C CNN
 F 1 "VCC" V 5900 6750 50  0000 C CNN
 F 2 "" H 5900 6550 50  0001 C CNN
@@
 $EndComp
 $Comp
-L VCC #PWR017
+L VCC #PWR10
 U 1 1 5AE8FC74
 P 2200 7300
-F 0 "#PWR017" H 2200 7150 50  0001 C CNN
+F 0 "#PWR10" H 2200 7150 50  0001 C CNN
 F 1 "VCC" V 2200 7500 50  0000 C CNN
 F 2 "" H 2200 7300 50  0001 C CNN
@@
 $EndComp
 $Comp
-L VCC #PWR018
+L VCC #PWR21
 U 1 1 5AE90B83
 P 5100 5750
-F 0 "#PWR018" H 5100 5600 50  0001 C CNN
+F 0 "#PWR21" H 5100 5600 50  0001 C CNN
 F 1 "VCC" V 5100 5950 50  0000 C CNN
 F 2 "" H 5100 5750 50  0001 C CNN
@@
 $EndComp
 $Comp
-L GND #PWR019
+L GND #PWR16
 U 1 1 5AE92C60
 P 4350 5950
-F 0 "#PWR019" H 4350 5700 50  0001 C CNN
+F 0 "#PWR16" H 4350 5700 50  0001 C CNN
 F 1 "GND" H 4350 5800 50  0000 C CNN
 F 2 "" H 4350 5950 50  0001 C CNN
@@
 $EndComp
 $Comp
-L GND #PWR020
+L GND #PWR17
 U 1 1 5AE92E0F
 P 4650 5950
-F 0 "#PWR020" H 4650 5700 50  0001 C CNN
+F 0 "#PWR17" H 4650 5700 50  0001 C CNN
 F 1 "GND" H 4650 5800 50  0000 C CNN
 F 2 "" H 4650 5950 50  0001 C CNN
@@
 $EndComp
 $Comp
-L +5V #PWR021
+L +5V #PWR24
 U 1 1 5AE94A9D
 P 5950 5450
-F 0 "#PWR021" H 5950 5300 50  0001 C CNN
+F 0 "#PWR24" H 5950 5300 50  0001 C CNN
 F 1 "+5V" V 6050 5500 50  0000 C CNN
 F 2 "" H 5950 5450 50  0001 C CNN
@@
 $EndComp
 $Comp
-L GND #PWR022
+L GND #PWR25
 U 1 1 5AE95087
 P 5950 5950
-F 0 "#PWR022" H 5950 5700 50  0001 C CNN
+F 0 "#PWR25" H 5950 5700 50  0001 C CNN
 F 1 "GND" V 5950 5750 50  0000 C CNN
 F 2 "" H 5950 5950 50  0001 C CNN
@@
 $EndComp
 $Comp
-L GND #PWR023
+L GND #PWR9
 U 1 1 5AE8857D
 P 1900 5400
-F 0 "#PWR023" H 1900 5150 50  0001 C CNN
+F 0 "#PWR9" H 1900 5150 50  0001 C CNN
 F 1 "GND" H 1900 5250 50  0000 C CNN
 F 2 "" H 1900 5400 50  0001 C CNN
@@
 Connection ~ 1100 5100
 $Comp
-L GND #PWR024
+L GND #PWR2
 U 1 1 5AE88AE3
 P 1100 5300
-F 0 "#PWR024" H 1100 5050 50  0001 C CNN
+F 0 "#PWR2" H 1100 5050 50  0001 C CNN
 F 1 "GND" H 1100 5150 50  0000 C CNN
 F 2 "" H 1100 5300 50  0001 C CNN
@@
 LIN
 $Comp
-L GND #PWR025
+L GND #PWR14
 U 1 1 5AE8F68F
 P 3250 6050
-F 0 "#PWR025" H 3250 5800 50  0001 C CNN
+F 0 "#PWR14" H 3250 5800 50  0001 C CNN
 F 1 "GND" H 3250 5900 50  0000 C CNN
 F 2 "" H 3250 6050 50  0001 C CNN
@@
 	1    0    0    -1
 $EndComp
+$Comp
+L AP1117-18 U2
+U 1 1 5B01A13D
+P 1450 5100
+F 0 "U2" H 1300 5225 50  0000 C CNN
+F 1 "AP1117-18" H 1450 5225 50  0000 L CNN
+F 2 "TO_SOT_Packages_SMD:SOT-223-3Lead_TabPin2" H 1450 5300 50  0001 C CNN
+F 3 "" H 1550 4850 50  0001 C CNN
+	1    1450 5100
+	1    0    0    -1
+$EndComp
