File: 3g_dcdc_usb_hub_board/3g_dcdc_usb_hub_board.sch (KiCad schematic (older format))
At the start: 30 parts, among them J1 G2116, J2 Conn_01x04, U1 DC_DC_BREAKOUT, U2 GL850G, Y1 Crystal

Commit message: Finished the GL850G-based USB hub&DCDC board
Parts:
- removed C6, C7: C_Small, Capacitors_SMD:C_0603, symbol C_Small
- removed RN1: R_Pack04, Resistors_SMD:R_Array_Convex_4x0603, symbol R_Pack04
- removed U2: GL850G, Housings_SSOP:SSOP-28_3.9x9.9mm_Pitch0.635mm, symbol GL850G
- added C10, C11, C12, C6, C7: C, Capacitors_SMD:C_0603, symbol C
- added JP1: MVC, footprints:GS2_SMALL, symbol Jumper_NO_Small
- added TP10: UB+, Measurement_Points:Measurement_Point_Round-SMD-Pad_Small, symbol TEST
- added TP9: UB-, Measurement_Points:Measurement_Point_Round-SMD-Pad_Small, symbol TEST
- added U2: FE1.1s, Housings_SSOP:SSOP-28_3.9x9.9mm_Pitch0.635mm, symbol FE1.1s
- R4: value 680R -> 2K7
Connections:
- net +3V3: now also C10.2, C6.2, C7.2, U2.13 (VD33), U2.17 (XRSTJ), U2.18 (V18), U2.19 (BUSJ), U2.21 (V33_O), U2.26 (OVCJ)
- net +5V: now also C12.2, JP1.1, U2.20 (V5); no longer J2.4 (Pin_4)
- net GND: now also R4.2, C10.1, C11.1, C12.1, C6.1, C7.1, U2.1 (VSS); no longer R4.1
- net UA+: now also U2.7 (DP3)
- net UA-: now also U2.6 (DM3)
- net UE+: now also U2.11 (DP1)
- net UE-: now also U2.10 (DM1)
- net UG+: now also U2.5 (DP4)
- net UG-: now also U2.4 (DM4)
- net UIN+: now also U2.16 (DPU)
- net UIN-: now also U2.15 (DMU)
- net at J1.3 (P3), J1.4 (P4): now also R5.2
- net at Y1.2: now also U2.3 (XIN)
- net at Y1.1: now also U2.2 (XOUT)
- new net: J2.4 (Pin_4), JP1.2
- new net: R4.1, U2.14 (REXT)
- new net +1V8: C11.2, U2.12 (VD18_O), U2.28 (VD18)
- new net UB+: TP10.1, U2.9 (DP2)
- new net UB-: TP9.1, U2.8 (DM2)
- no-connect marks 6 -> 5
Other:
- moved on the sheet: D1, J2, R1, TP1, TP2, TP3, TP4, TP5, TP6, TP7, TP8, Y1
