File: 24xx_i2c_so8_programming/24xx_i2c_programming.sch (KiCad schematic (older format))
At the start: 11 parts, among them J1 EXPANSION_BOTTOM, J2 A0, J3 A1, J4 A2, J5 WP, U1 24LC00

Commit message: Giving the 24xx SO8 board a new name, changing the passive footprints, adding +- on the silkscreen
Parts:
- C1: footprint Capacitors_SMD:C_0603_HandSoldering -> Capacitors_SMD:C_0805_HandSoldering
- R1, R2, R3, R4: footprint Resistors_SMD:R_0603_HandSoldering -> Resistors_SMD:R_0805_HandSoldering
Changed lines of the file:
@@
 F 0 "C1" H 3625 4250 50  0000 L CNN
 F 1 "C" H 3625 4050 50  0000 L CNN
-F 2 "Capacitors_SMD:C_0603_HandSoldering" H 3638 4000 50  0001 C CNN
+F 2 "Capacitors_SMD:C_0805_HandSoldering" H 3638 4000 50  0001 C CNN
 F 3 "" H 3600 4150 50  0001 C CNN
 	1    3600 4150
@@
 F 0 "R1" V 4700 4200 50  0000 L CNN
 F 1 "10K" V 4650 4150 50  0000 L CNN
-F 2 "Resistors_SMD:R_0603_HandSoldering" H 4700 4250 50  0001 C CNN
+F 2 "Resistors_SMD:R_0805_HandSoldering" H 4700 4250 50  0001 C CNN
 F 3 "" H 4700 4250 50  0001 C CNN
 	1    4700 4250
@@
 F 0 "R3" V 5000 4200 50  0000 L CNN
 F 1 "10K" V 4950 4150 50  0000 L CNN
-F 2 "Resistors_SMD:R_0603_HandSoldering" H 5000 4250 50  0001 C CNN
+F 2 "Resistors_SMD:R_0805_HandSoldering" H 5000 4250 50  0001 C CNN
 F 3 "" H 5000 4250 50  0001 C CNN
 	1    5000 4250
@@
 F 0 "R2" V 4850 4200 50  0000 L CNN
 F 1 "10K" V 4800 4150 50  0000 L CNN
-F 2 "Resistors_SMD:R_0603_HandSoldering" H 4850 4250 50  0001 C CNN
+F 2 "Resistors_SMD:R_0805_HandSoldering" H 4850 4250 50  0001 C CNN
 F 3 "" H 4850 4250 50  0001 C CNN
 	1    4850 4250
@@
 F 0 "R4" V 5950 4200 50  0000 L CNN
 F 1 "10K" V 5900 4150 50  0000 L CNN
-F 2 "Resistors_SMD:R_0603_HandSoldering" H 5950 4250 50  0001 C CNN
+F 2 "Resistors_SMD:R_0805_HandSoldering" H 5950 4250 50  0001 C CNN
 F 3 "" H 5950 4250 50  0001 C CNN
 	1    5950 4250
