File: dock_connection_board_gamma/dock_connection_board.kicad_pcb (KiCad board)
At the start: 2 copper layers, 33 x 25.4 mm, 14 parts, among them J1 USBO, J2 USBI, J3 CHG, J4 I2CI, J5 AUXI, J6 ANI, J7 I2CO, U1 24LC32

Commit message: Dock board v1.1 - fixing the dock board outline and positioning
Parts:
- J2: moved to B.Cu
- moved J2 0.07 mm to (137.1, 114.2), turned to 0 degrees
- moved J4 0.05 mm to (124.5, 104.1)
- moved J5 0.05 mm to (124.5, 121.9)
Other:
- board text added: "Dock adapter for ZP Gamma, by CRImier, v1.0"
- board text removed: "Dock adapter for ZP Delta, by CRImier, v1.0"
Changed lines of the file:
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@@
   (general
     (links 32)
-    (no_connects 5)
+    (no_connects 0)
     (area 112.954999 102.794999 146.125001 128.345001)
     (thickness 1.6)
@@
     )
   )
-  (module Pin_Headers:Pin_Header_Straight_1x04_Pitch2.54mm (layer F.Cu)
-    (at 137.16 114.3 180)
+  (module Pin_Headers:Pin_Header_Straight_1x04_Pitch2.54mm (layer B.Cu)
+    (at 137.1092 114.2492)
     (descr "Through hole straight pin header, 1x04, 2.54mm pitch, single row")
     (tags "Through hole pin header THT 1x04 2.54mm single row")
-    (fp_text reference J2 (at 0 -2.33 180) (layer F.SilkS) hide
-      (effects (font (size 1 1) (thickness 0.15)))
-    )
-    (fp_text value USBI (at 0 9.95 180) (layer F.Fab) hide
-      (effects (font (size 1 1) (thickness 0.15)))
-    )
-    (fp_line (start -0.635 -1.27) (end 1.27 -1.27) (layer F.Fab) (width 0.1))
-    (fp_line (start 1.27 -1.27) (end 1.27 8.89) (layer F.Fab) (width 0.1))
-    (fp_line (start 1.27 8.89) (end -1.27 8.89) (layer F.Fab) (width 0.1))
-    (fp_line (start -1.27 8.89) (end -1.27 -0.635) (layer F.Fab) (width 0.1))
-    (fp_line (start -1.27 -0.635) (end -0.635 -1.27) (layer F.Fab) (width 0.1))
-    (fp_line (start -1.33 8.95) (end 1.33 8.95) (layer F.SilkS) (width 0.12))
-    (fp_line (start -1.33 1.27) (end -1.33 8.95) (layer F.SilkS) (width 0.12))
-    (fp_line (start 1.33 1.27) (end 1.33 8.95) (layer F.SilkS) (width 0.12))
-    (fp_line (start -1.33 1.27) (end 1.33 1.27) (layer F.SilkS) (width 0.12))
-    (fp_line (start -1.33 0) (end -1.33 -1.33) (layer F.SilkS) (width 0.12))
-    (fp_line (start -1.33 -1.33) (end 0 -1.33) (layer F.SilkS) (width 0.12))
-    (fp_line (start -1.8 -1.8) (end -1.8 9.4) (layer F.CrtYd) (width 0.05))
-    (fp_line (start -1.8 9.4) (end 1.8 9.4) (layer F.CrtYd) (width 0.05))
-    (fp_line (start 1.8 9.4) (end 1.8 -1.8) (layer F.CrtYd) (width 0.05))
-    (fp_line (start 1.8 -1.8) (end -1.8 -1.8) (layer F.CrtYd) (width 0.05))
-    (fp_text user %R (at 0 3.81 270) (layer F.Fab)
-      (effects (font (size 1 1) (thickness 0.15)))
-    )
-    (pad 1 thru_hole rect (at 0 0 180) (size 1.7 1.7) (drill 1) (layers *.Cu *.Mask)
+    (fp_text reference J2 (at 0 2.33) (layer B.SilkS) hide
+      (effects (font (size 1 1) (thickness 0.15)) (justify mirror))
+    )
+    (fp_text value USBI (at 0 -9.95) (layer B.Fab) hide
+      (effects (font (size 1 1) (thickness 0.15)) (justify mirror))
+    )
+    (fp_line (start -0.635 1.27) (end 1.27 1.27) (layer B.Fab) (width 0.1))
+    (fp_line (start 1.27 1.27) (end 1.27 -8.89) (layer B.Fab) (width 0.1))
+    (fp_line (start 1.27 -8.89) (end -1.27 -8.89) (layer B.Fab) (width 0.1))
+    (fp_line (start -1.27 -8.89) (end -1.27 0.635) (layer B.Fab) (width 0.1))
+    (fp_line (start -1.27 0.635) (end -0.635 1.27) (layer B.Fab) (width 0.1))
+    (fp_line (start -1.33 -8.95) (end 1.33 -8.95) (layer B.SilkS) (width 0.12))
+    (fp_line (start -1.33 -1.27) (end -1.33 -8.95) (layer B.SilkS) (width 0.12))
+    (fp_line (start 1.33 -1.27) (end 1.33 -8.95) (layer B.SilkS) (width 0.12))
+    (fp_line (start -1.33 -1.27) (end 1.33 -1.27) (layer B.SilkS) (width 0.12))
+    (fp_line (start -1.33 0) (end -1.33 1.33) (layer B.SilkS) (width 0.12))
+    (fp_line (start -1.33 1.33) (end 0 1.33) (layer B.SilkS) (width 0.12))
+    (fp_line (start -1.8 1.8) (end -1.8 -9.4) (layer B.CrtYd) (width 0.05))
+    (fp_line (start -1.8 -9.4) (end 1.8 -9.4) (layer B.CrtYd) (width 0.05))
+    (fp_line (start 1.8 -9.4) (end 1.8 1.8) (layer B.CrtYd) (width 0.05))
+    (fp_line (start 1.8 1.8) (end -1.8 1.8) (layer B.CrtYd) (width 0.05))
+    (fp_text user %R (at 0 -3.81 270) (layer B.Fab)
+      (effects (font (size 1 1) (thickness 0.15)) (justify mirror))
+    )
+    (pad 1 thru_hole rect (at 0 0) (size 1.7 1.7) (drill 1) (layers *.Cu *.Mask)
       (net 6 "Net-(J2-Pad1)"))
-    (pad 2 thru_hole oval (at 0 2.54 180) (size 1.7 1.7) (drill 1) (layers *.Cu *.Mask)
+    (pad 2 thru_hole oval (at 0 -2.54) (size 1.7 1.7) (drill 1) (layers *.Cu *.Mask)
       (net 4 D-))
-    (pad 3 thru_hole oval (at 0 5.08 180) (size 1.7 1.7) (drill 1) (layers *.Cu *.Mask)
+    (pad 3 thru_hole oval (at 0 -5.08) (size 1.7 1.7) (drill 1) (layers *.Cu *.Mask)
       (net 5 D+))
-    (pad 4 thru_hole oval (at 0 7.62 180) (size 1.7 1.7) (drill 1) (layers *.Cu *.Mask)
+    (pad 4 thru_hole oval (at 0 -7.62) (size 1.7 1.7) (drill 1) (layers *.Cu *.Mask)
       (net 2 GND))
     (model ${KISYS3DMOD}/Pin_Headers.3dshapes/Pin_Header_Straight_1x04_Pitch2.54mm.wrl
@@
   )
   (module Pin_Headers:Pin_Header_Straight_1x05_Pitch2.54mm (layer F.Cu)
-    (at 124.46 104.14)
+    (at 124.46 104.0892)
     (descr "Through hole straight pin header, 1x05, 2.54mm pitch, single row")
     (tags "Through hole pin header THT 1x05 2.54mm single row")
@@
     (pad 5 thru_hole oval (at 0 10.16) (size 1.7 1.7) (drill 1) (layers *.Cu *.Mask)
       (net 1 +3V3))
-    (model ${KISYS3DMOD}/Pin_Headers.3dshapes/Pin_Header_Straight_1x05_Pitch2.54mm.wrl
-      (at (xyz 0 0 0))
+    (model Pin_Headers.3dshapes/Pin_Header_Angled_1x05_Pitch2.54mm.wrl
+      (at (xyz 0 -0.4 0))
       (scale (xyz 1 1 1))
-      (rotate (xyz 0 0 0))
+      (rotate (xyz 0 0 180))
     )
   )
   (module Pin_Headers:Pin_Header_Straight_1x03_Pitch2.54mm (layer F.Cu)
-    (at 124.46 121.92)
+    (at 124.46 121.8692)
     (descr "Through hole straight pin header, 1x03, 2.54mm pitch, single row")
     (tags "Through hole pin header THT 1x03 2.54mm single row")
@@
     (pad 3 thru_hole oval (at 0 5.08) (size 1.7 1.7) (drill 1) (layers *.Cu *.Mask)
       (net 7 CHG))
-    (model ${KISYS3DMOD}/Pin_Headers.3dshapes/Pin_Header_Straight_1x03_Pitch2.54mm.wrl
-      (at (xyz 0 0 0))
+    (model Pin_Headers.3dshapes/Pin_Header_Angled_1x03_Pitch2.54mm.wrl
+      (at (xyz 0 -0.2 0))
       (scale (xyz 1 1 1))
-      (rotate (xyz 0 0 0))
+      (rotate (xyz 0 0 180))
     )
   )
@@
     (pad 3 thru_hole oval (at 0 5.08 180) (size 1.7 1.7) (drill 1) (layers *.Cu *.Mask)
       (net 1 +3V3))
-    (model ${KISYS3DMOD}/Pin_Headers.3dshapes/Pin_Header_Straight_1x03_Pitch2.54mm.wrl
-      (at (xyz 0 0 0))
-      (scale (xyz 1 1 1))
-      (rotate (xyz 0 0 0))
-    )
   )
   (module Pin_Headers:Pin_Header_Straight_1x05_Pitch2.54mm (layer F.Cu)
@@
     (pad 5 thru_hole oval (at 0 10.16 90) (size 1.7 1.7) (drill 1) (layers *.Cu *.Mask)
       (net 2 GND))
-    (model ${KISYS3DMOD}/Pin_Headers.3dshapes/Pin_Header_Straight_1x05_Pitch2.54mm.wrl
-      (at (xyz 0 0 0))
-      (scale (xyz 1 1 1))
-      (rotate (xyz 0 0 0))
-    )
   )
   (module Connect:GS2 (layer F.Cu)
@@
     (pad 5 thru_hole oval (at 0 10.16) (size 1.7 1.7) (drill 1) (layers *.Cu *.Mask)
       (net 7 CHG))
-    (model ${KISYS3DMOD}/Pin_Headers.3dshapes/Pin_Header_Straight_1x05_Pitch2.54mm.wrl
-      (at (xyz 0 0 0))
-      (scale (xyz 1 1 1))
-      (rotate (xyz 0 0 0))
-    )
   )
   (module Terminal_Blocks:TerminalBlock_bornier-2_P5.08mm (layer F.Cu)
@@
   (gr_circle (center 136.433283 118.11) (end 137.616123 119.126) (layer Edge.Cuts) (width 0.15))
   (gr_circle (center 127.980717 115.57) (end 129.163557 116.586) (layer Edge.Cuts) (width 0.15))
-  (gr_text "Dock\nadapter for ZP Delta,\nby CRImier, v1.0" (at 125.984 120.396) (layer F.SilkS)
+  (gr_text "Dock\nadapter for ZP Gamma,\nby CRImier, v1.0" (at 125.984 120.396) (layer F.SilkS)
     (effects (font (size 1 1) (thickness 0.2)) (justify left))
   )
