File: sh1106_1.3_spi_breakout/sh1106_1.3_spi_breakout.sch (KiCad schematic (older format))
At the start: 20 parts, among them J1 OLED_HEADER, J2 OLED_PANEL, Q1 Q_PMOS_GSD

Commit message: Small routing adjustments
Parts:
- J1: symbol CONN_01X06 -> Conn_01x06
- J2: symbol CONN_01X30 -> Conn_01x30
Changed lines of the file:
@@
 EESchema Schematic File Version 2
+LIBS:sh1106_1.3_spi_breakout-rescue
 LIBS:power
 LIBS:device
@@
 LIBS:contrib
 LIBS:valves
-LIBS:sh1106_1.3_spi_display-cache
 EELAYER 25 0
 EELAYER END
@@
 $EndDescr
 $Comp
-L CONN_01X30 J2
+L Conn_01x30 J2
 U 1 1 59933012
-P 5550 3550
-F 0 "J2" H 5550 5100 50  0000 C CNN
-F 1 "OLED_PANEL" V 5650 3550 50  0000 C CNN
-F 2 "libs:FPC_30" H 5550 3550 50  0001 C CNN
-F 3 "" H 5550 3550 50  0001 C CNN
-	1    5550 3550
+P 5550 3500
+F 0 "J2" H 5550 5050 50  0000 C CNN
+F 1 "OLED_PANEL" V 5650 3500 50  0000 C CNN
+F 2 "libs:FPC_30" H 5550 3500 50  0001 C CNN
+F 3 "" H 5550 3500 50  0001 C CNN
+	1    5550 3500
 	1    0    0    -1
 $EndComp
@@
 $EndComp
 $Comp
-L CONN_01X06 J1
+L Conn_01x06 J1
 U 1 1 5993459F
 P 2650 3550
@@
 L GND #PWR015
 U 1 1 599345E6
-P 2450 3400
-F 0 "#PWR015" H 2450 3150 50  0001 C CNN
-F 1 "GND" V 2450 3200 50  0000 C CNN
-F 2 "" H 2450 3400 50  0001 C CNN
-F 3 "" H 2450 3400 50  0001 C CNN
-	1    2450 3400
-	0    1    1    0
-$EndComp
-Text GLabel 2450 3500 0    60   Input ~ 0
+P 2450 3450
+F 0 "#PWR015" H 2450 3200 50  0001 C CNN
+F 1 "GND" V 2450 3250 50  0000 C CNN
+F 2 "" H 2450 3450 50  0001 C CNN
+F 3 "" H 2450 3450 50  0001 C CNN
+	1    2450 3450
+	0    1    1    0
+$EndComp
+Text GLabel 2450 3550 0    60   Input ~ 0
 CLK
-Text GLabel 2450 3600 0    60   Input ~ 0
+Text GLabel 2450 3650 0    60   Input ~ 0
 MOSI
-Text GLabel 2450 3700 0    60   Input ~ 0
+Text GLabel 2450 3750 0    60   Input ~ 0
 CS
-Text GLabel 2450 3800 0    60   Input ~ 0
+Text GLabel 2450 3850 0    60   Input ~ 0
 DC
 $Comp
@@
 L VCC #PWR037
 U 1 1 59961EEB
-P 2450 3300
-F 0 "#PWR037" H 2450 3150 50  0001 C CNN
-F 1 "VCC" V 2450 3500 50  0000 C CNN
-F 2 "" H 2450 3300 50  0001 C CNN
-F 3 "" H 2450 3300 50  0001 C CNN
-	1    2450 3300
+P 2450 3350
+F 0 "#PWR037" H 2450 3200 50  0001 C CNN
+F 1 "VCC" V 2450 3550 50  0000 C CNN
+F 2 "" H 2450 3350 50  0001 C CNN
+F 3 "" H 2450 3350 50  0001 C CNN
+	1    2450 3350
 	0    -1   -1   0
 $EndComp

Commit message: Fixing the FPC connector on the SH1106 PCB - v1.2
Parts:
- added FID1, FID2, FID3, FID4: FID, Fiducials:Fiducial_0.75mm_Dia_1.5mm_Outer, symbol TEST
- C1: value C_Small -> 10uF
- C2, C4, C5, C6, C8: value C_Small -> 1uF
- C3: value C_Small -> 4.7uF
- C7: value C_Small -> 100nF
- D1: value D_Small -> 1N4148
- J2: footprint libs:FPC_30 -> libs:FPC_30_correct
- Q1: value Q_PMOS_GSD -> CJ2305
- R1, R2, R3, R4, R5, R8: value R_Small -> 10K
- R6: value R_Small -> 390K
- R7: value R_Small -> 1K
Connections:
- net +3V3: now also D1.1 (K), J2.22 (Pin_22), J2.25 (Pin_25); no longer D1.2 (A), J2.6 (Pin_6), J2.9 (Pin_9)
- net CLK: now also J2.13 (Pin_13); no longer J2.18 (Pin_18)
- net CS: now also J2.18 (Pin_18); no longer J2.13 (Pin_13)
- net DC: now also J2.16 (Pin_16); no longer J2.15 (Pin_15)
- net GND: now also J2.14 (Pin_14), J2.15 (Pin_15), J2.19 (Pin_19), J2.2 (Pin_2), J2.6 (Pin_6), J2.9 (Pin_9); no longer J2.12 (Pin_12), J2.16 (Pin_16), J2.17 (Pin_17), J2.22 (Pin_22), J2.25 (Pin_25), J2.29 (Pin_29)
- net MOSI: now also J2.12 (Pin_12); no longer J2.19 (Pin_19)
- net RESET: now also D1.2 (A), J2.17 (Pin_17); no longer D1.1 (K), J2.14 (Pin_14)
- net at C2.2: now also J2.29 (Pin_29); no longer J2.2 (Pin_2)
- net at J2.26 (Pin_26): now also C6.1; no longer R6.1
- net at J2.27 (Pin_27): now also C6.2; no longer C3.1
- net at C4.1, C5.1: now also J2.3 (Pin_3); no longer J2.28 (Pin_28)
- net at C2.1: now also J2.28 (Pin_28); no longer J2.3 (Pin_3)
- net at J2.4 (Pin_4): now also C3.1; no longer C6.2
- net at J2.5 (Pin_5): now also R6.1; no longer C6.1
Changed lines of the file:
@@
 LIBS:contrib
 LIBS:valves
+LIBS:sh1106_1.3_spi_breakout-cache
 EELAYER 25 0
 EELAYER END
@@
 L Conn_01x30 J2
 U 1 1 59933012
-P 5550 3500
-F 0 "J2" H 5550 5050 50  0000 C CNN
-F 1 "OLED_PANEL" V 5650 3500 50  0000 C CNN
-F 2 "libs:FPC_30" H 5550 3500 50  0001 C CNN
-F 3 "" H 5550 3500 50  0001 C CNN
-	1    5550 3500
-	1    0    0    -1
+P 5550 3600
+F 0 "J2" H 5550 5150 50  0000 C CNN
+F 1 "OLED_PANEL" V 5650 3600 50  0000 C CNN
+F 2 "libs:FPC_30_correct" H 5550 3600 50  0001 C CNN
+F 3 "" H 5550 3600 50  0001 C CNN
+	1    5550 3600
+	1    0    0    1
 $EndComp
 $Comp
@@
 P 4700 4900
 F 0 "C4" V 4750 4950 50  0000 L CNN
-F 1 "C_Small" V 4600 4750 50  0000 L CNN
+F 1 "1uF" V 4600 4750 50  0000 L CNN
 F 2 "Capacitors_SMD:C_0805" H 4700 4900 50  0001 C CNN
 F 3 "" H 4700 4900 50  0001 C CNN
@@
 P 4700 4700
 F 0 "C3" V 4750 4750 50  0000 L CNN
-F 1 "C_Small" V 4600 4550 50  0000 L CNN
+F 1 "4.7uF" V 4600 4550 50  0000 L CNN
 F 2 "Capacitors_SMD:C_0805" H 4700 4700 50  0001 C CNN
 F 3 "" H 4700 4700 50  0001 C CNN
@@
 P 4700 4500
 F 0 "R6" V 4700 4450 50  0000 L CNN
-F 1 "R_Small" V 4600 4350 50  0000 L CNN
+F 1 "390K" V 4600 4350 50  0000 L CNN
 F 2 "Resistors_SMD:R_0805" H 4700 4500 50  0001 C CNN
 F 3 "" H 4700 4500 50  0001 C CNN
@@
 P 4500 2250
 F 0 "C2" H 4550 2350 50  0000 L CNN
-F 1 "C_Small" H 4100 2250 50  0000 L CNN
+F 1 "1uF" H 4100 2250 50  0000 L CNN
 F 2 "Capacitors_SMD:C_0805" H 4500 2250 50  0001 C CNN
 F 3 "" H 4500 2250 50  0001 C CNN
@@
 P 4800 2450
 F 0 "C6" H 4850 2550 50  0000 L CNN
-F 1 "C_Small" H 4400 2450 50  0000 L CNN
+F 1 "1uF" H 4400 2450 50  0000 L CNN
 F 2 "Capacitors_SMD:C_0805" H 4800 2450 50  0001 C CNN
 F 3 "" H 4800 2450 50  0001 C CNN
@@
 P 3850 3400
 F 0 "C1" H 3750 3500 50  0000 L CNN
-F 1 "C_Small" V 3950 3150 50  0000 L CNN
+F 1 "10uF" H 3950 3400 50  0000 L CNN
 F 2 "Capacitors_SMD:C_0805" H 3850 3400 50  0001 C CNN
 F 3 "" H 3850 3400 50  0001 C CNN
@@
 P 3850 3100
 F 0 "R5" V 3850 3050 50  0000 L CNN
-F 1 "R_Small" V 3950 3050 50  0000 L CNN
+F 1 "10K" H 3950 3100 50  0000 L CNN
 F 2 "Resistors_SMD:R_0805" H 3850 3100 50  0001 C CNN
 F 3 "" H 3850 3100 50  0001 C CNN
@@
 P 3650 3100
 F 0 "D1" H 3600 3180 50  0000 L CNN
-F 1 "D_Small" H 3500 3020 50  0000 L CNN
+F 1 "1N4148" H 3500 3020 50  0000 L CNN
 F 2 "Diodes_SMD:D_0805" V 3650 3100 50  0001 C CNN
 F 3 "" V 3650 3100 50  0001 C CNN
 	1    3650 3100
-	0    -1   -1   0
+	0    1    1    0
 $EndComp
 Wire Wire Line
@@
 P 3650 4550
 F 0 "R4" V 3650 4500 50  0000 L CNN
-F 1 "R_Small" V 3700 4400 50  0000 L CNN
+F 1 "10K" V 3700 4400 50  0000 L CNN
 F 2 "Resistors_SMD:R_0805" H 3650 4550 50  0001 C CNN
 F 3 "" H 3650 4550 50  0001 C CNN
@@
 P 3650 4350
 F 0 "R3" V 3650 4300 50  0000 L CNN
-F 1 "R_Small" V 3700 4200 50  0000 L CNN
+F 1 "10K" V 3700 4200 50  0000 L CNN
 F 2 "Resistors_SMD:R_0805" H 3650 4350 50  0001 C CNN
 F 3 "" H 3650 4350 50  0001 C CNN
@@
 P 3650 4150
 F 0 "R2" V 3650 4100 50  0000 L CNN
-F 1 "R_Small" V 3700 4000 50  0000 L CNN
+F 1 "10K" V 3700 4000 50  0000 L CNN
 F 2 "Resistors_SMD:R_0805" H 3650 4150 50  0001 C CNN
 F 3 "" H 3650 4150 50  0001 C CNN
@@
 P 3650 3950
 F 0 "R1" V 3650 3900 50  0000 L CNN
-F 1 "R_Small" V 3700 3800 50  0000 L CNN
+F 1 "10K" V 3700 3800 50  0000 L CNN
 F 2 "Resistors_SMD:R_0805" H 3650 3950 50  0001 C CNN
 F 3 "" H 3650 3950 50  0001 C CNN
@@
 P 4700 5100
 F 0 "C5" V 4750 5150 50  0000 L CNN
-F 1 "C_Small" V 4600 4950 50  0000 L CNN
+F 1 "1uF" V 4600 4950 50  0000 L CNN
 F 2 "Capacitors_SMD:C_0805" H 4700 5100 50  0001 C CNN
 F 3 "" H 4700 5100 50  0001 C CNN
@@
 P 2350 4250
 F 0 "C7" V 2400 4300 50  0000 L CNN
-F 1 "C_Small" V 2250 4100 50  0000 L CNN
+F 1 "100nF" V 2250 4100 50  0000 L CNN
 F 2 "Capacitors_SMD:C_0805" H 2350 4250 50  0001 C CNN
 F 3 "" H 2350 4250 50  0001 C CNN
@@
 P 3050 2100
 F 0 "Q1" V 2900 1900 50  0000 L CNN
-F 1 "Q_PMOS_GSD" V 3350 1900 50  0000 L CNN
+F 1 "CJ2305" V 3350 1900 50  0000 L CNN
 F 2 "TO_SOT_Packages_SMD:SOT-23" H 3250 2200 50  0001 C CNN
 F 3 "" H 3050 2100 50  0001 C CNN
@@
 P 2750 4250
 F 0 "C8" V 2800 4300 50  0000 L CNN
-F 1 "C_Small" V 2650 4100 50  0000 L CNN
+F 1 "1uF" V 2650 4100 50  0000 L CNN
 F 2 "Capacitors_SMD:C_0805" H 2750 4250 50  0001 C CNN
 F 3 "" H 2750 4250 50  0001 C CNN
@@
 P 3300 2150
 F 0 "R8" V 3300 2100 50  0000 L CNN
-F 1 "R_Small" V 3400 2100 50  0000 L CNN
+F 1 "10K" V 3400 2100 50  0000 L CNN
 F 2 "Resistors_SMD:R_0805" H 3300 2150 50  0001 C CNN
 F 3 "" H 3300 2150 50  0001 C CNN
@@
 P 3050 2500
 F 0 "R7" V 3050 2450 50  0000 L CNN
-F 1 "R_Small" V 3150 2300 50  0000 L CNN
+F 1 "1K" V 3150 2300 50  0000 L CNN
 F 2 "Resistors_SMD:R_0805" H 3050 2500 50  0001 C CNN
 F 3 "" H 3050 2500 50  0001 C CNN
@@
 	0    -1   -1   0
 $EndComp
+$Comp
+L TEST FID1
+U 1 1 5B48BD61
+P 1850 1350
+F 0 "FID1" H 1850 1650 50  0000 C BNN
+F 1 "FID" H 1850 1600 50  0000 C CNN
+F 2 "Fiducials:Fiducial_0.75mm_Dia_1.5mm_Outer" H 1850 1350 50  0001 C CNN
+F 3 "" H 1850 1350 50  0001 C CNN
+	1    1850 1350
+	1    0    0    -1
+$EndComp
+$Comp
+L TEST FID2
+U 1 1 5B48C097
+P 2050 1350
+F 0 "FID2" H 2050 1650 50  0000 C BNN
+F 1 "FID" H 2050 1600 50  0000 C CNN
+F 2 "Fiducials:Fiducial_0.75mm_Dia_1.5mm_Outer" H 2050 1350 50  0001 C CNN
+F 3 "" H 2050 1350 50  0001 C CNN
+	1    2050 1350
+	1    0    0    -1
+$EndComp
+$Comp
+L TEST FID3
+U 1 1 5B48C0FD
+P 2250 1350
+F 0 "FID3" H 2250 1650 50  0000 C BNN
+F 1 "FID" H 2250 1600 50  0000 C CNN
+F 2 "Fiducials:Fiducial_0.75mm_Dia_1.5mm_Outer" H 2250 1350 50  0001 C CNN
+F 3 "" H 2250 1350 50  0001 C CNN
+	1    2250 1350
+	1    0    0    -1
+$EndComp
+$Comp
+L TEST FID4
+U 1 1 5B48C15A
+P 2450 1350
+F 0 "FID4" H 2450 1650 50  0000 C BNN
+F 1 "FID" H 2450 1600 50  0000 C CNN
+F 2 "Fiducials:Fiducial_0.75mm_Dia_1.5mm_Outer" H 2450 1350 50  0001 C CNN
+F 3 "" H 2450 1350 50  0001 C CNN
+	1    2450 1350
+	1    0    0    -1
+$EndComp
 $EndSCHEMATC
