File: attinyx5_programming/attinyx5_programming.sch (KiCad schematic (older format))
At the start: 6 parts, among them P2 CONN_01X06, U1 ATTINY85-20SU, Y1 Crystal

Commit message: v1.1 of ATTiny PCB - fixing the ATTiny FP, adding an additional ATTIny to track the RST pin
Parts:
- added C4: C_Small, Capacitors_SMD:C_0805, symbol C_Small
- added CON1: AVR-ISP-6, Pin_Headers:Pin_Header_Straight_2x03_Pitch1.27mm_SMD, symbol AVR-ISP-6
- added JP1: Jumper, footprints:GS2_SMALL, symbol Jumper
- added R1: 10K, Resistors_SMD:R_0805, symbol R_Small
- added U2: ATTINY13-20SU, Housings_SOIC:SSO-8_6.8x5.9mm_Pitch1.27mm_Clearance7mm, symbol ATTINY13-20SU
- C1, C2, C3: footprint Capacitors_SMD:C_0805_HandSoldering -> Capacitors_SMD:C_0805
- U1: footprint Housings_SOIC:SOIC-8_3.9x4.9mm_Pitch1.27mm -> Housings_SOIC:SSO-8_6.8x5.9mm_Pitch1.27mm_Clearance7mm
Connections:
- net +3V3: now also C4.1, CON1.2, R1.2, U2.8 (VCC)
- net CLK: now also CON1.3, U2.7 (PB2(SCK/ADC1/T0/PCINT2))
- net CS: now also JP1.2, U2.3 (PB4(ADC2/PCINT4)); no longer U1.1 (PB5(~RESET~/dW/ADC0/PCINT5))
- net GND: now also C4.2, CON1.6, U2.4 (GND)
- net MISO: now also CON1.1, U2.6 (PB1(MISO/AIN1/OC0B/INT0/PCINT1))
- net MOSI: now also CON1.4, U2.5 (PB0(MOSI/AIN0/OC0A/PCINT0))
- new net: CON1.5, R1.1, U2.1 (PB5(~RESET~/ADC0/PCINT5/dW))
- new net RST: JP1.1, U1.1 (PB5(~RESET~/dW/ADC0/PCINT5)), U2.2 (PB3(CLKI/ADC3/PCINT3))
Changed lines of the file:
@@
 F 0 "C1" H 5110 3220 50  0000 L CNN
 F 1 "C_Small" H 5110 3070 50  0000 L CNN
-F 2 "Capacitors_SMD:C_0805_HandSoldering" H 5100 3150 50  0001 C CNN
+F 2 "Capacitors_SMD:C_0805" H 5100 3150 50  0001 C CNN
 F 3 "" H 5100 3150 50  0000 C CNN
 	1    5100 3150
@@
 $EndComp
 $Comp
-L +3.3V #PWR7
+L +3.3V #PWR14
 U 1 1 590E98A4
 P 5850 3350
-F 0 "#PWR7" H 5850 3200 50  0001 C CNN
+F 0 "#PWR14" H 5850 3200 50  0001 C CNN
 F 1 "+3.3V" V 5850 3600 50  0000 C CNN
 F 2 "" H 5850 3350 50  0000 C CNN
@@
 $EndComp
 $Comp
-L GND #PWR8
+L GND #PWR15
 U 1 1 590E98E4
 P 5850 3450
-F 0 "#PWR8" H 5850 3200 50  0001 C CNN
+F 0 "#PWR15" H 5850 3200 50  0001 C CNN
 F 1 "GND" V 5850 3250 50  0000 C CNN
 F 2 "" H 5850 3450 50  0000 C CNN
@@
 CS
 $Comp
-L +3.3V #PWR5
+L +3.3V #PWR12
 U 1 1 590E9977
 P 5100 3050
-F 0 "#PWR5" H 5100 2900 50  0001 C CNN
+F 0 "#PWR12" H 5100 2900 50  0001 C CNN
 F 1 "+3.3V" H 5100 3200 50  0000 C CNN
 F 2 "" H 5100 3050 50  0000 C CNN
@@
 $EndComp
 $Comp
-L GND #PWR6
+L GND #PWR13
 U 1 1 590E99A1
 P 5100 3250
-F 0 "#PWR6" H 5100 3000 50  0001 C CNN
+F 0 "#PWR13" H 5100 3000 50  0001 C CNN
 F 1 "GND" H 5100 3100 50  0000 C CNN
 F 2 "" H 5100 3250 50  0000 C CNN
@@
 $EndComp
 Text GLabel 1750 3400 0    60   Input ~ 0
-CS
+RST
 Text GLabel 1750 3100 0    60   Input ~ 0
 CLK
@@
 F 0 "U1" H 1950 3550 50  0000 C CNN
 F 1 "ATTINY85-20SU" H 4100 2750 50  0000 C CNN
-F 2 "Housings_SOIC:SOIC-8_3.9x4.9mm_Pitch1.27mm" H 4050 3150 50  0001 C CIN
+F 2 "Housings_SOIC:SSO-8_6.8x5.9mm_Pitch1.27mm_Clearance7mm" H 4050 3150 50  0001 C CIN
 F 3 "" H 3100 3150 50  0001 C CNN
 	1    3100 3150
@@
 $EndComp
 $Comp
-L +3.3V #PWR3
+L +3.3V #PWR8
 U 1 1 5AEEE196
 P 4450 2900
-F 0 "#PWR3" H 4450 2750 50  0001 C CNN
+F 0 "#PWR8" H 4450 2750 50  0001 C CNN
 F 1 "+3.3V" V 4450 3150 50  0000 C CNN
 F 2 "" H 4450 2900 50  0000 C CNN
@@
 F 0 "C2" H 910 3170 50  0000 L CNN
 F 1 "C_Small" H 910 3020 50  0000 L CNN
-F 2 "Capacitors_SMD:C_0805_HandSoldering" H 900 3100 50  0001 C CNN
+F 2 "Capacitors_SMD:C_0805" H 900 3100 50  0001 C CNN
 F 3 "" H 900 3100 50  0001 C CNN
 	1    900  3100
@@
 F 0 "C3" H 910 3470 50  0000 L CNN
 F 1 "C_Small" H 910 3320 50  0000 L CNN
-F 2 "Capacitors_SMD:C_0805_HandSoldering" H 900 3400 50  0001 C CNN
+F 2 "Capacitors_SMD:C_0805" H 900 3400 50  0001 C CNN
 F 3 "" H 900 3400 50  0001 C CNN
 	1    900  3400
@@
 Connection ~ 1250 3400
 $Comp
-L GND #PWR4
+L GND #PWR9
 U 1 1 5AEEE46E
 P 4450 3400
-F 0 "#PWR4" H 4450 3150 50  0001 C CNN
+F 0 "#PWR9" H 4450 3150 50  0001 C CNN
 F 1 "GND" V 4450 3200 50  0000 C CNN
 F 2 "" H 4450 3400 50  0000 C CNN
@@
 	0    -1   -1   0
 $EndComp
+$Comp
+L ATTINY13-20SU U2
+U 1 1 5C3B4737
+P 3350 900
+F 0 "U2" H 2550 1300 50  0000 C CNN
+F 1 "ATTINY13-20SU" H 4000 500 50  0000 C CNN
+F 2 "Housings_SOIC:SSO-8_6.8x5.9mm_Pitch1.27mm_Clearance7mm" H 4000 900 50  0001 C CIN
+F 3 "" H 2550 1250 50  0001 C CNN
+	1    3350 900
+	1    0    0    -1
+$EndComp
+$Comp
+L +3.3V #PWR6
+U 1 1 5C3B479F
+P 4350 650
+F 0 "#PWR6" H 4350 500 50  0001 C CNN
+F 1 "+3.3V" V 4350 900 50  0000 C CNN
+F 2 "" H 4350 650 50  0000 C CNN
+F 3 "" H 4350 650 50  0000 C CNN
+	1    4350 650
+	0    1    1    0
+$EndComp
+$Comp
+L GND #PWR7
+U 1 1 5C3B47A5
+P 4350 1150
+F 0 "#PWR7" H 4350 900 50  0001 C CNN
+F 1 "GND" V 4350 950 50  0000 C CNN
+F 2 "" H 4350 1150 50  0000 C CNN
+F 3 "" H 4350 1150 50  0000 C CNN
+	1    4350 1150
+	0    -1   -1   0
+$EndComp
+Text GLabel 2350 1050 0    60   Input ~ 0
+CS
+Text GLabel 2350 950  0    60   Input ~ 0
+RST
+Text GLabel 2350 850  0    60   Input ~ 0
+CLK
+$Comp
+L C_Small C4
+U 1 1 5C3B4836
+P 5050 900
+F 0 "C4" H 5060 970 50  0000 L CNN
+F 1 "C_Small" H 5060 820 50  0000 L CNN
+F 2 "Capacitors_SMD:C_0805" H 5050 900 50  0001 C CNN
+F 3 "" H 5050 900 50  0000 C CNN
+	1    5050 900
+	1    0    0    -1
+$EndComp
+$Comp
+L +3.3V #PWR10
+U 1 1 5C3B483C
+P 5050 800
+F 0 "#PWR10" H 5050 650 50  0001 C CNN
+F 1 "+3.3V" H 5050 950 50  0000 C CNN
+F 2 "" H 5050 800 50  0000 C CNN
+F 3 "" H 5050 800 50  0000 C CNN
+	1    5050 800
+	1    0    0    -1
+$EndComp
+$Comp
+L GND #PWR11
+U 1 1 5C3B4842
+P 5050 1000
+F 0 "#PWR11" H 5050 750 50  0001 C CNN
+F 1 "GND" H 5050 850 50  0000 C CNN
+F 2 "" H 5050 1000 50  0000 C CNN
+F 3 "" H 5050 1000 50  0000 C CNN
+	1    5050 1000
+	1    0    0    -1
+$EndComp
+$Comp
+L R_Small R1
+U 1 1 5C3B48F3
+P 2100 1150
+F 0 "R1" V 2200 1100 50  0000 L CNN
+F 1 "10K" V 2100 1100 50  0000 L CNN
+F 2 "Resistors_SMD:R_0805" H 2100 1150 50  0001 C CNN
+F 3 "" H 2100 1150 50  0001 C CNN
+	1    2100 1150
+	0    1    1    0
+$EndComp
+$Comp
+L +3.3V #PWR3
+U 1 1 5C3B4AE3
+P 2000 1150
+F 0 "#PWR3" H 2000 1000 50  0001 C CNN
+F 1 "+3.3V" V 2000 1400 50  0000 C CNN
+F 2 "" H 2000 1150 50  0000 C CNN
+F 3 "" H 2000 1150 50  0000 C CNN
+	1    2000 1150
+	0    -1   -1   0
+$EndComp
+$Comp
+L Jumper JP1
+U 1 1 5C3B4B4A
+P 1150 2400
+F 0 "JP1" H 1150 2550 50  0000 C CNN
+F 1 "Jumper" H 1150 2320 50  0000 C CNN
+F 2 "footprints:GS2_SMALL" H 1150 2400 50  0001 C CNN
+F 3 "" H 1150 2400 50  0001 C CNN
+	1    1150 2400
+	1    0    0    -1
+$EndComp
+Text GLabel 1450 2400 2    60   Input ~ 0
+CS
+Text GLabel 850  2400 0    60   Input ~ 0
+RST
+Text GLabel 2350 650  0    60   Input ~ 0
+MOSI
+Text GLabel 2350 750  0    60   Input ~ 0
+MISO
+$Comp
+L AVR-ISP-6 CON1
+U 1 1 5C3B534C
+P 3000 1600
+F 0 "CON1" H 2895 1840 50  0000 C CNN
+F 1 "AVR-ISP-6" H 2735 1370 50  0000 L BNN
+F 2 "Pin_Headers:Pin_Header_Straight_2x03_Pitch1.27mm_SMD" V 2480 1640 50  0001 C CNN
+F 3 "" H 2975 1600 50  0001 C CNN
+	1    3000 1600
+	1    0    0    -1
+$EndComp
+Text GLabel 3500 1600 2    60   Input ~ 0
+MOSI
+Wire Wire Line
+	2200 1150 2350 1150
+Wire Wire Line
+	2300 1150 2300 1700
+Wire Wire Line
+	2300 1700 2850 1700
+Connection ~ 2300 1150
+Text GLabel 2600 1600 0    60   Input ~ 0
+CLK
+Wire Wire Line
+	2850 1600 2600 1600
+Text GLabel 2600 1500 0    60   Input ~ 0
+MISO
+Wire Wire Line
+	2850 1500 2600 1500
+$Comp
+L +3.3V #PWR4
+U 1 1 5C3B5802
+P 3500 1500
+F 0 "#PWR4" H 3500 1350 50  0001 C CNN
+F 1 "+3.3V" V 3500 1750 50  0000 C CNN
+F 2 "" H 3500 1500 50  0000 C CNN
+F 3 "" H 3500 1500 50  0000 C CNN
+	1    3500 1500
+	0    1    1    0
+$EndComp
+Wire Wire Line
+	3100 1500 3500 1500
+Wire Wire Line
+	3500 1600 3100 1600
+$Comp
+L GND #PWR5
+U 1 1 5C3B5886
+P 3500 1700
+F 0 "#PWR5" H 3500 1450 50  0001 C CNN
+F 1 "GND" V 3500 1500 50  0000 C CNN
+F 2 "" H 3500 1700 50  0000 C CNN
+F 3 "" H 3500 1700 50  0000 C CNN
+	1    3500 1700
+	0    -1   -1   0
+$EndComp
+Wire Wire Line
+	3100 1700 3500 1700
 $EndSCHEMATC
