File: osd3358_cpu_board/osd3358_cpu_board.kicad_pcb (KiCad board)
At the start: 2 copper layers, 12 parts, among them J1 Conn_02x20_Odd_Even, J2 USB_OTG, J3 USB_OTG, U1 OSD3358-512M-BSM, U2 MICROSD

Commit message: Today's work
Parts:
- added C1, C4: 100nF, Capacitors_SMD:C_0402, F.Cu at (140.0, 81.8)
- added C2, C3: 18pF, Capacitors_SMD:C_0402, F.Cu at (140.0, 81.8)
- added D1: PWR, LEDs:LED_0805, F.Cu at (140.0, 81.8)
- added D2: LED0, LEDs:LED_0805, F.Cu at (140.0, 81.8)
- added D3: LED1, LEDs:LED_0805, F.Cu at (140.0, 81.8)
- added D4: LED2, LEDs:LED_0805, F.Cu at (140.0, 81.8)
- added D5: LED3, LEDs:LED_0805, F.Cu at (140.0, 81.8)
- added J5: USB_PCTL, Pin_Headers:Pin_Header_Straight_1x05_Pitch1.27mm, F.Cu at (148.8, 82.2)
- added J6: AIN_1.8V, Pin_Headers:Pin_Header_Straight_1x05_Pitch1.27mm, F.Cu at (148.8, 72.3)
- added L1: 120R, Capacitors_SMD:C_0603, F.Cu at (140.0, 81.8)
- added L2: Ferrite_Bead_Small, Capacitors_SMD:C_0603, F.Cu at (140.0, 81.8)
- added R3, R4, R5: 10K, Resistors_SMD:R_0402, F.Cu at (140.0, 81.8)
- added R6: 0R, Resistors_SMD:R_0402, F.Cu at (140.0, 81.8)
- added RN5, RN6, RN7, RN8: 10K, Resistors_SMD:R_Array_Concave_4x0402, F.Cu at (140.0, 81.8)
- added RN9: 1K, Resistors_SMD:R_Array_Concave_4x0402, F.Cu at (140.0, 81.8)
- added SW1: SW_Push, Buttons_Switches_SMD:SW_SPST_B3U-1000P, F.Cu at (140.0, 81.8)
- added U3: 74AHC1G07, TO_SOT_Packages_SMD:SOT-353_SC-70-5, F.Cu at (140.0, 81.8)
- added Y1: Crystal, osd3358_cpu_board:CRYSTAL_5X3.2MM, F.Cu at (140.0, 81.8)
- J2: value USB_OTG -> USB_IN
- J3: value USB_OTG -> USB_OUT
- RN1, RN2: value R_Pack04 -> 10K
Connections:
- J2 pad 6: GND -> Net-(J2-Pad6)
- J3 pad 6: GND -> Net-(J2-Pad6)
- U1 pad A7: (no net) -> VREFP
- U1 pad A9: (no net) -> VREFN
- U1 pad B7: (no net) -> VREFP
- U1 pad B9: (no net) -> VREFN
- U1 pad C10: (no net) -> Net-(U1-PadC10)
- U1 pad C11: (no net) -> Net-(U1-PadC11)
- U1 pad C7: (no net) -> Net-(J6-Pad1)
- U1 pad C8: (no net) -> Net-(J6-Pad2)
- U1 pad C9: (no net) -> Net-(J6-Pad4)
- U1 pad D10: (no net) -> Net-(U1-PadC10)
- U1 pad D11: (no net) -> Net-(U1-PadC11)
- U1 pad D3: (no net) -> TRST
- U1 pad D4: (no net) -> Net-(U1-PadD4)
- U1 pad D6: (no net) -> Net-(U1-PadD6)
- U1 pad D7: (no net) -> Net-(U1-PadD6)
- U1 pad D8: (no net) -> GND
- U1 pad D9: (no net) -> GND
- U1 pad E10: (no net) -> GND
- U1 pad E11: (no net) -> GND
- U1 pad E12: (no net) -> GND
- U1 pad E4: (no net) -> Net-(U1-PadD4)
- U1 pad E5: (no net) -> GND
- U1 pad E6: (no net) -> GND
- U1 pad E7: (no net) -> GND
- U1 pad E8: (no net) -> GND
- U1 pad E9: (no net) -> GND
- U1 pad F10: (no net) -> +1V8
- U1 pad F11: (no net) -> +3.3VADC
- U1 pad F12: (no net) -> GND
- U1 pad F5: (no net) -> GND
- U1 pad F6: (no net) -> +3.3VA
- U1 pad F7: (no net) -> +3.3VA
- U1 pad F8: (no net) -> +3.3VP
- U1 pad F9: (no net) -> +3.3VP
- U1 pad G1: (no net) -> /LCD2
- U1 pad G10: (no net) -> +1V8
- U1 pad G11: (no net) -> +3.3VADC
- U1 pad G12: (no net) -> GND
- U1 pad G2: (no net) -> /LCD1
- U1 pad G3: (no net) -> /LCD0
- U1 pad G5: (no net) -> GND
- U1 pad G6: (no net) -> +3.3VA
- U1 pad G7: (no net) -> +3.3VA
- U1 pad G8: (no net) -> +3.3VP
- U1 pad G9: (no net) -> +3.3VP
- U1 pad H1: (no net) -> /LCD5
- U1 pad H10: (no net) -> +1V8
- U1 pad H11: (no net) -> +1V8
- U1 pad H12: (no net) -> GND
- U1 pad H13: (no net) -> GND
- U1 pad H16: (no net) -> SD_EN
- U1 pad H2: (no net) -> /LCD4
- U1 pad H3: (no net) -> /LCD3
- U1 pad H4: (no net) -> GND
- U1 pad H5: (no net) -> GND
- U1 pad H7: (no net) -> +3.3VP
- U1 pad H8: (no net) -> +3.3VP
- U1 pad H9: (no net) -> +3.3VP
- U1 pad J1: (no net) -> /LCD8
- U1 pad J10: (no net) -> +1V8
- U1 pad J11: (no net) -> +1V8
- U1 pad J12: (no net) -> GND
- U1 pad J13: (no net) -> GND
- U1 pad J15: (no net) -> Net-(J5-Pad4)
- U1 pad J16: Net-(J2-Pad1) -> +5VD
- U1 pad J2: (no net) -> /LCD7
- U1 pad J3: (no net) -> /LCD6
- U1 pad J4: (no net) -> GND
- U1 pad J5: (no net) -> GND
- U1 pad J7: (no net) -> +3.3VP
- U1 pad J8: (no net) -> +3.3VP
- U1 pad J9: (no net) -> +3.3VP
- U1 pad K1: (no net) -> /LCD11
- U1 pad K10: (no net) -> +1V8
- U1 pad K11: (no net) -> VMEM
- U1 pad K12: (no net) -> GND
- U1 pad K13: (no net) -> Net-(J5-Pad5)
- U1 pad K2: (no net) -> /LCD10
- U1 pad K3: (no net) -> /LCD9
- U1 pad K5: (no net) -> GND
- U1 pad K6: (no net) -> +5VP
- U1 pad K7: (no net) -> +5VP
- U1 pad K8: (no net) -> +3.3VP
- U1 pad K9: (no net) -> +3.3VP
- U1 pad L1: (no net) -> /LCD14
- U1 pad L10: (no net) -> +1V8
- U1 pad L11: (no net) -> VMEM
- U1 pad L12: (no net) -> GND
- U1 pad L13: (no net) -> Net-(J5-Pad1)
- U1 pad L2: (no net) -> /LCD13
- U1 pad L3: (no net) -> /LCD12
- U1 pad L4: (no net) -> Net-(U1-PadL4)
- U1 pad L5: (no net) -> GND
- U1 pad L6: (no net) -> +5VP
- U1 pad L7: (no net) -> +5VP
- U1 pad L8: (no net) -> +3.3VP
- U1 pad L9: (no net) -> +3.3VP
- U1 pad M10: (no net) -> GND
- U1 pad M11: (no net) -> GND
- U1 pad M12: (no net) -> GND
- U1 pad M14: (no net) -> Net-(J5-Pad2)
- U1 pad M16: (no net) -> Net-(R3-Pad1)
- U1 pad M2: (no net) -> /EEP_WP
- U1 pad M3: (no net) -> /LCD15
- U1 pad M4: (no net) -> Net-(U1-PadL4)
- U1 pad M5: (no net) -> GND
- U1 pad M6: (no net) -> GND
- U1 pad M7: (no net) -> GND
- U1 pad M8: (no net) -> GND
- U1 pad M9: (no net) -> GND
- U1 pad N10: (no net) -> Net-(U1-PadN10)
- U1 pad N11: (no net) -> Net-(U1-PadN10)
- U1 pad N12: (no net) -> /PMIC_PGOOD
- U1 pad N13: (no net) -> Net-(J6-Pad5)
- U1 pad N15: (no net) -> Net-(C2-Pad2)
- U1 pad N16: (no net) -> Net-(C3-Pad1)
- U1 pad N3: (no net) -> /EEP_WP
- U1 pad N4: (no net) -> Net-(TP2-Pad1)
- U1 pad N5: (no net) -> Net-(TP2-Pad1)
- U1 pad N7: (no net) -> +BATT
- U1 pad N8: (no net) -> GND
- U1 pad N9: (no net) -> GND
- U1 pad P10: (no net) -> +VDC
- U1 pad P11: (no net) -> /PMIC_PGOOD
- U1 pad P13: (no net) -> LED0
- U1 pad P14: (no net) -> LED3
- U1 pad P16: (no net) -> Net-(C2-Pad1)
- U1 pad P8: (no net) -> +BATT
- U1 pad P9: (no net) -> +5VD
- U1 pad R10: (no net) -> +VDC
- U1 pad R11: (no net) -> /~RESET
- U1 pad R14: (no net) -> LED2
- U1 pad R8: (no net) -> +BATT
- U1 pad R9: (no net) -> +5VD
- U1 pad T10: (no net) -> +VDC
- U1 pad T11: (no net) -> Net-(SW1-Pad2)
- U1 pad T14: (no net) -> LED1
- U1 pad T8: (no net) -> +BATT
- U1 pad T9: (no net) -> +5VD
