File: osd3358_cpu_board/osd3358_cpu_board.sch (KiCad schematic (older format))
At the start: 11 parts, among them J1 Conn_02x20_Odd_Even, J2 USB_OTG, J3 USB_OTG, U1 OSD3358-512M-BSM, U2 MICROSD

Commit message: Today's work
Parts:
- added C1, C4: 100nF, Capacitors_SMD:C_0402, symbol C_Small
- added C2, C3: 18pF, Capacitors_SMD:C_0402, symbol C_Small
- added D1: PWR, LEDs:LED_0805, symbol LED
- added D2: LED0, LEDs:LED_0805, symbol LED
- added D3: LED1, LEDs:LED_0805, symbol LED
- added D4: LED2, LEDs:LED_0805, symbol LED
- added D5: LED3, LEDs:LED_0805, symbol LED
- added J4: JTAG, symbol Conn_01x09
- added J5: USB_PCTL, Pin_Headers:Pin_Header_Straight_1x05_Pitch1.27mm, symbol Conn_01x05
- added J6: AIN_1.8V, Pin_Headers:Pin_Header_Straight_1x05_Pitch1.27mm, symbol Conn_01x05
- added L1: 120R, Capacitors_SMD:C_0603, symbol Ferrite_Bead_Small
- added L2: Ferrite_Bead_Small, Capacitors_SMD:C_0603, symbol Ferrite_Bead_Small
- added R3, R4, R5: 10K, Resistors_SMD:R_0402, symbol R_Small
- added R6: 0R, Resistors_SMD:R_0402, symbol R_Small
- added RN5, RN6, RN7, RN8: 10K, Resistors_SMD:R_Array_Concave_4x0402, symbol R_Pack04
- added RN9: 1K, Resistors_SMD:R_Array_Concave_4x0402, symbol R_Pack04
- added SW1: SW_Push, Buttons_Switches_SMD:SW_SPST_B3U-1000P, symbol SW_Push
- added TP1: EEP_WP, symbol TEST
- added TP10: VDDS_PLL, symbol TEST
- added TP2: LDO_PGOOD, symbol TEST
- added TP3: JT_E0, symbol TEST
- added TP4: JT_E1, symbol TEST
- added TP5: VREF+, symbol TEST
- added TP6: VREF-, symbol TEST
- added TP7: VDDS_DDR, symbol TEST
- added TP8: VDD_CORE, symbol TEST
- added TP9: VDD_MPU, symbol TEST
- added U3: 74AHC1G07, TO_SOT_Packages_SMD:SOT-353_SC-70-5, symbol 74AHC1G04
- added Y1: Crystal, osd3358_cpu_board:CRYSTAL_5X3.2MM, symbol Crystal
- J2: value USB_OTG -> USB_IN
- J3: value USB_OTG -> USB_OUT
- RN1, RN2: value R_Pack04 -> 10K
Connections:
- net +3.3VA: now also U1.F6 (SYS_VDD1_3P3V), U1.F7 (SYS_VDD1_3P3V), U1.G6 (SYS_VDD1_3P3V), U1.G7 (SYS_VDD1_3P3V), RN5.5 (R4.2), RN6.8 (R1.2), RN8.6 (R3.2)
- net GND: now also U1.D8 (DGND), U1.D9 (DGND), U1.E10 (DGND), U1.E11 (DGND), U1.E12 (DGND), U1.E5 (DGND), U1.E6 (DGND), U1.E7 (DGND), U1.E8 (DGND), U1.E9 (DGND), U1.F12 (DGND), U1.F5 (DGND), U1.G12 (DGND), U1.G5 (DGND), U1.H12 (DGND), U1.H13 (DGND), U1.H4 (DGND), U1.H5 (DGND), U1.J12 (DGND), U1.J13 (DGND), U1.J4 (DGND), U1.J5 (DGND), U1.K12 (DGND), U1.K5 (DGND), U1.L12 (DGND), U1.L5 (DGND), U1.M10 (DGND), U1.M11 (DGND), U1.M12 (DGND), U1.M5 (DGND), U1.M6 (DGND), U1.M7 (DGND), U1.M8 (DGND), U1.M9 (DGND), U1.N8 (DGND), U1.N9 (DGND), C1.2, D2.1 (K), D3.1 (K), D4.1 (K), D5.1 (K), J4.4 (Pin_4), J4.7 (Pin_7), J4.9 (Pin_9), J5.3 (Pin_3), J6.3 (Pin_3), L2.2, R3.2, R4.1, R5.1, RN5.6 (R3.2), RN5.7 (R2.2), RN5.8 (R1.2), RN6.5 (R4.2), RN6.6 (R3.2), RN6.7 (R2.2), RN7.5 (R4.2), RN7.6 (R3.2), RN7.7 (R2.2), RN7.8 (R1.2), RN8.5 (R4.2), RN8.7 (R2.2), RN8.8 (R1.2), SW1.1, U3.3 (GND); no longer J2.6 (Shield), J3.6 (Shield)
- net ID_SD: now also R6.2
- net SD_EN: now also R6.1
- net EEP_WP: now reaches U1.N3 (GPMC_BEN0_CLE)
- net EEP_WP: now also U1.M2 (EEPROM_WP), TP1.1
- net LED0: now reaches U1.P13 (GPMC_A5)
- net LED0: now also RN9.1 (R1.1)
- net LED3: now reaches U1.P14 (GPMC_A8)
- net LED3: now also RN9.4 (R4.1)
- net LED2: now reaches U1.R14 (GPMC_A7)
- net LED2: now also RN9.3 (R3.1)
- net LED1: now reaches U1.T14 (GPMC_A6)
- net LED1: now also RN9.2 (R2.1)
- net at U1.C10 (I2C0_SCL): now also U1.D10 (PMIC_SCL)
- net at U1.C11 (I2C0_SDA): now also U1.D11 (PMIC_SDA)
- net at U1.D4 (EXTINTN): now also U1.E4 (PMIC_NINT)
- net +1V8: now reaches U1.F10 (SYS_VDD_1P8V)
- net +1V8: now also U1.G10 (SYS_VDD_1P8V), U1.H10 (SYS_VDD_1P8V), U1.H11 (SYS_VDD_1P8V), U1.J10 (SYS_VDD_1P8V), U1.J11 (SYS_VDD_1P8V), U1.K10 (SYS_VDD_1P8V), U1.L10 (SYS_VDD_1P8V)
- net +3.3VADC: now reaches U1.F11 (SYS_VDD2_3P3V)
- net +3.3VADC: now also U1.G11 (SYS_VDD2_3P3V), D1.2 (A)
- net +3.3VP: now reaches U1.F8 (SYS_VDD3_3P3V)
- net +3.3VP: now also U1.F9 (VDDSHV4), U1.G8 (SYS_VDD3_3P3V), U1.G9 (VDDSHV5), U1.H7 (SYS_VDD3_3P3V), U1.H8 (SYS_VDD3_3P3V), U1.H9 (VDDSHV6), U1.J7 (SYS_VDD3_3P3V), U1.J8 (SYS_VDD3_3P3V), U1.J9 (VDDSHV1), U1.K8 (SYS_VDD3_3P3V), U1.K9 (VDDSHV2), U1.L8 (SYS_VDD3_3P3V), U1.L9 (VDDSHV3)
- net VMEM: now reaches U1.K11 (SYS_RTC_1P8V)
- net VMEM: now also U1.L11 (SYS_RTC_1P8V), C1.1, U3.5 (VCC)
- net +5VP: now reaches U1.K6 (SYS_VOUT)
- net +5VP: now also U1.K7 (SYS_VOUT), U1.L6 (SYS_VOUT), U1.L7 (SYS_VOUT)
- net at U1.L4 (PMIC_NWAKEUP): now also U1.M4 (EXT_WAKEUP)
- net at U1.M16 (RTC_KALDO_ENN): now also R3.1
- net at U1.N10 (PMIC_POWER_EN): now also U1.N11 (PMIC_PWR_EN)
- net PMIC_PGOOD: now reaches U1.N12 (PMIC_PGOOD)
- net PMIC_PGOOD: now also U1.P11 (PWRONRSTN), U3.2
- net at U1.N4 (PMIC_LDO_PGOOD): now also U1.N5 (RTC_PWRONRSTN), TP2.1
- net TS: now reaches U1.N6 (PMIC_TS)
- net +BATT: now reaches U1.N7 (PMIC_BAT_SENSE)
- net +BATT: now also U1.P8 (VIN_BAT), U1.R8 (VIN_BAT), U1.T8 (VIN_BAT)
- net +VDC: now reaches U1.P10 (VIN_AC)
- net +VDC: now also U1.R10 (VIN_AC), U1.T10 (VIN_AC)
- net +5VD: now reaches U1.P9 (VIN_USB)
- net +5VD: now also U1.J16 (USB0_VBUS), U1.R9 (VIN_USB), U1.T9 (VIN_USB), L1.2
- net ~RESET: now reaches U1.R11 (WARMRSTN)
- net ~RESET: now also J4.1 (Pin_1), U3.4
- net at U1.T11 (PMIC_PB_IN): now also SW1.2
- net VREFP: now reaches U1.A7 (SYS_ADC_1P8V)
- net VREFP: now also U1.B7 (VREFP), C4.1, TP5.1
- net VREFN: now reaches U1.A9 (AGND_ADC)
- net VREFN: now also U1.B9 (VREFN), C4.2, TP6.1
- net TDI: now reaches U1.C1 (TDI)
- net TDI: now also J4.3 (Pin_3)
- net TDO: now reaches U1.C2 (TDO)
- net TDO: now also J4.5 (Pin_5)
- net at U1.C7 (AIN4): now also J6.1 (Pin_1)
- net at U1.C8 (AIN5): now also J6.2 (Pin_2)
- net at U1.C9 (AIN6): now also J6.4 (Pin_4)
- net TCK: now reaches U1.D1 (TCK)
- net TCK: now also J4.8 (Pin_8)
- net TMS: now reaches U1.D2 (TMS)
- net TMS: now also J4.6 (Pin_6)
- net TRST: now reaches U1.D3 (TRSTN)
- net TRST: now also J4.2 (Pin_2), R5.2
- net at U1.D6 (PMIC_MUX_OUT): now also U1.D7 (AIN7)
- net at U1.E2 (EMU0): now also TP3.1
- net at U1.E3 (EMU1): now also TP4.1
- net at U1.J15 (USB0_DRVVBUS): now also J5.4 (Pin_4)
- net at J2.1 (VBUS): now also L1.1; no longer U1.J16 (USB0_VBUS)
- net at U1.K13 (USB0_CE): now also J5.5 (Pin_5)
- net at U1.L13 (USB1_CE): now also J5.1 (Pin_1)
- net at U1.M14 (USB1_DRVVBUS): now also J5.2 (Pin_2)
- net at U1.N13 (PMIC_MUX_IN): now also J6.5 (Pin_5)
- net at U1.N15 (OSC0_GND): now also C2.2, C3.2
- net at U1.N16 (OSC0_OUT): now also C3.1, Y1.2
- net at U1.P16 (OSC0_IN): now also C2.1, Y1.1
- net LCD2: now reaches U1.G1 (LCD_DATA2)
- net LCD2: now also RN5.3 (R3.1)
- net LCD1: now reaches U1.G2 (LCD_DATA1)
- net LCD1: now also RN5.2 (R2.1)
- net LCD0: now reaches U1.G3 (LCD_DATA0)
- net LCD0: now also RN5.1 (R1.1)
- net LCD5: now reaches U1.H1 (LCD_DATA5)
- net LCD5: now also RN6.2 (R2.1)
- net LCD4: now reaches U1.H2 (LCD_DATA4)
- net LCD4: now also RN6.1 (R1.1)
- net LCD3: now reaches U1.H3 (LCD_DATA3)
- net LCD3: now also RN5.4 (R4.1)
- net LCD8: now reaches U1.J1 (LCD_DATA8)
- net LCD8: now also RN7.1 (R1.1)
- net LCD7: now reaches U1.J2 (LCD_DATA7)
- net LCD7: now also RN6.4 (R4.1)
- net LCD6: now reaches U1.J3 (LCD_DATA6)
- net LCD6: now also RN6.3 (R3.1)
- net LCD11: now reaches U1.K1 (LCD_DATA11)
- net LCD11: now also RN7.4 (R4.1)
- net LCD10: now reaches U1.K2 (LCD_DATA10)
- net LCD10: now also RN7.3 (R3.1)
- net LCD9: now reaches U1.K3 (LCD_DATA9)
- net LCD9: now also RN7.2 (R2.1)
- net LCD14: now reaches U1.L1 (LCD_DATA14)
- net LCD14: now also RN8.3 (R3.1)
- net LCD13: now reaches U1.L2 (LCD_DATA13)
- net LCD13: now also RN8.2 (R2.1)
- net LCD12: now reaches U1.L3 (LCD_DATA12)
- net LCD12: now also RN8.1 (R1.1)
- net LCD15: now reaches U1.M3 (LCD_DATA15)
- net LCD15: now also RN8.4 (R4.1)
- net at U1.F13 (VDD_MPU): now also TP9.1
- net at U1.F4 (VDDS_DDR): now also TP7.1
- net at U1.G13 (VDDS_PLL): now also TP10.1
- net at U1.G4 (VDD_CORE): now also TP8.1
- new net: J2.6 (Shield), J3.6 (Shield), L2.1
- new net: D1.1 (K), R4.2
- new net: D5.2 (A), RN9.5 (R4.2)
- new net: D4.2 (A), RN9.6 (R3.2)
- new net: D3.2 (A), RN9.7 (R2.2)
- new net: D2.2 (A), RN9.8 (R1.2)
- no-connect marks 52 -> 60
